File: Sensors.sch (KiCad schematic (older format))
At the start: 19 parts, among them U2 ICM-20602, U3 BMP388, U5 BMM150, U7 ICM-42605, U8 BMI088

Commit message: working
Other:
- moved on the sheet: C13, C14, R1, R2, U7
Changed lines of the file:
@@
 Wire Wire Line
 	2800 1950 2800 2500
-Text GLabel 2900 1200 2    50   Input ~ 0
-SENSORS_3V3
 Wire Wire Line
 	1800 1450 1900 1450
@@
 L power:GND #PWR0108
 U 1 1 61BD2100
-P 1500 4750
-F 0 "#PWR0108" H 1500 4500 50  0001 C CNN
-F 1 "GND" H 1505 4577 50  0000 C CNN
-F 2 "" H 1500 4750 50  0001 C CNN
-F 3 "" H 1500 4750 50  0001 C CNN
-	1    1500 4750
-	1    0    0    -1
-$EndComp
-Text GLabel 1100 4750 0    50   Input ~ 0
-SENSORS_3V3
-Wire Wire Line
-	1500 4450 1200 4450
-Connection ~ 1500 4450
-Wire Wire Line
-	1100 4750 1200 4750
-Wire Wire Line
-	1600 4450 1500 4450
+P 1550 4750
+F 0 "#PWR0108" H 1550 4500 50  0001 C CNN
+F 1 "GND" H 1555 4577 50  0000 C CNN
+F 2 "" H 1550 4750 50  0001 C CNN
+F 3 "" H 1550 4750 50  0001 C CNN
+	1    1550 4750
+	1    0    0    -1
+$EndComp
+Wire Wire Line
+	1550 4450 1250 4450
+Connection ~ 1550 4450
+Wire Wire Line
+	1600 4450 1550 4450
 Text Notes 450  3400 0    394  ~ 0
 BMP388
@@
 L Device:R R2
 U 1 1 61B9F3F5
-P 1200 4600
-F 0 "R2" H 1270 4646 50  0000 L CNN
-F 1 "DNP" H 1270 4555 50  0000 L CNN
-F 2 "Resistor_SMD:R_0402_1005Metric" V 1130 4600 50  0001 C CNN
-F 3 "~" H 1200 4600 50  0001 C CNN
-F 4 "~" H 1200 4600 50  0001 C CNN "Datasheet"
-F 5 "Resistor_SMD:R_0402_1005Metric" H 1200 4600 50  0001 C CNN "Footprint"
-F 6 "R2" H 1200 4600 50  0001 C CNN "Reference"
-F 7 "DNP" H 1200 4600 50  0001 C CNN "Value"
-	1    1200 4600
+P 1250 4600
+F 0 "R2" H 1320 4646 50  0000 L CNN
+F 1 "DNP" H 1320 4555 50  0000 L CNN
+F 2 "Resistor_SMD:R_0402_1005Metric" V 1180 4600 50  0001 C CNN
+F 3 "~" H 1250 4600 50  0001 C CNN
+F 4 "~" H 1250 4600 50  0001 C CNN "Datasheet"
+F 5 "Resistor_SMD:R_0402_1005Metric" H 1250 4600 50  0001 C CNN "Footprint"
+F 6 "R2" H 1250 4600 50  0001 C CNN "Reference"
+F 7 "DNP" H 1250 4600 50  0001 C CNN "Value"
+	1    1250 4600
 	1    0    0    -1
 $EndComp
@@
 L Device:R R1
 U 1 1 61B9BCC8
-P 1500 4600
-F 0 "R1" H 1570 4646 50  0000 L CNN
-F 1 "0R" H 1570 4555 50  0000 L CNN
-F 2 "Resistor_SMD:R_0402_1005Metric" V 1430 4600 50  0001 C CNN
-F 3 "~" H 1500 4600 50  0001 C CNN
-F 4 "~" H 1500 4600 50  0001 C CNN "Datasheet"
-F 5 "Resistor_SMD:R_0402_1005Metric" H 1500 4600 50  0001 C CNN "Footprint"
-F 6 "R1" H 1500 4600 50  0001 C CNN "Reference"
-F 7 "0R" H 1500 4600 50  0001 C CNN "Value"
-	1    1500 4600
+P 1550 4600
+F 0 "R1" H 1620 4646 50  0000 L CNN
+F 1 "0R" H 1620 4555 50  0000 L CNN
+F 2 "Resistor_SMD:R_0402_1005Metric" V 1480 4600 50  0001 C CNN
+F 3 "~" H 1550 4600 50  0001 C CNN
+F 4 "~" H 1550 4600 50  0001 C CNN "Datasheet"
+F 5 "Resistor_SMD:R_0402_1005Metric" H 1550 4600 50  0001 C CNN "Footprint"
+F 6 "R1" H 1550 4600 50  0001 C CNN "Reference"
+F 7 "0R" H 1550 4600 50  0001 C CNN "Value"
+	1    1550 4600
 	1    0    0    -1
 $EndComp
@@
 	1    0    0    -1
 $EndComp
-Text GLabel 3000 3750 2    50   Input ~ 0
-SENSORS_3V3
 Wire Notes Line
 	500  5000 500  2900
@@
 	1    0    0    -1
 $EndComp
-Text Notes 500  5550 0    394  ~ 0
-BMM155
 Wire Notes Line
 	500  5050 4000 5050
@@
 Wire Wire Line
 	1800 5750 1900 5750
-Text GLabel 2500 5750 2    50   Input ~ 0
-SENSORS_3V3
 Wire Wire Line
 	2500 5750 1900 5750
@@
 Wire Wire Line
 	2350 6250 2300 6250
-Text GLabel 3250 6250 2    50   Input ~ 0
-SENSORS_3V3
 $Comp
 L Device:C C6
@@
 Wire Notes Line
 	500  9250 500  6850
-Wire Wire Line
-	3350 8300 3350 8450
 $Comp
 L Device:C C13
 U 1 1 61C6DAF2
-P 3200 8300
-F 0 "C13" V 3350 8250 50  0000 L CNN
-F 1 "100nF" V 3300 8200 50  0000 L CNN
-F 2 "Capacitor_SMD:C_0402_1005Metric" H 3238 8150 50  0001 C CNN
-F 3 "~" H 3200 8300 50  0001 C CNN
-F 4 "~" H 3200 8300 50  0001 C CNN "Datasheet"
-F 5 "Capacitor_SMD:C_0402_1005Metric" H 3200 8300 50  0001 C CNN "Footprint"
-F 6 "C13" H 3200 8300 50  0001 C CNN "Reference"
-F 7 "100nF" H 3200 8300 50  0001 C CNN "Value"
-	1    3200 8300
+P 3150 8300
+F 0 "C13" V 3300 8250 50  0000 L CNN
+F 1 "100nF" V 3250 8200 50  0000 L CNN
+F 2 "Capacitor_SMD:C_0402_1005Metric" H 3188 8150 50  0001 C CNN
+F 3 "~" H 3150 8300 50  0001 C CNN
+F 4 "~" H 3150 8300 50  0001 C CNN "Datasheet"
+F 5 "Capacitor_SMD:C_0402_1005Metric" H 3150 8300 50  0001 C CNN "Footprint"
+F 6 "C13" H 3150 8300 50  0001 C CNN "Reference"
+F 7 "100nF" H 3150 8300 50  0001 C CNN "Value"
+	1    3150 8300
 	0    -1   -1   0
 $EndComp
 Wire Wire Line
-	3050 8300 3050 8200
+	3000 8300 3000 8200
 $Comp
 L Device:C C14
 U 1 1 61C6F18A
-P 3200 8600
-F 0 "C14" V 3350 8550 50  0000 L CNN
-F 1 "2.2uF" V 3400 8500 50  0000 L CNN
-F 2 "Capacitor_SMD:C_0402_1005Metric" H 3238 8450 50  0001 C CNN
-F 3 "~" H 3200 8600 50  0001 C CNN
-F 4 "~" H 3200 8600 50  0001 C CNN "Datasheet"
-F 5 "Capacitor_SMD:C_0402_1005Metric" H 3200 8600 50  0001 C CNN "Footprint"
-F 6 "C14" H 3200 8600 50  0001 C CNN "Reference"
-F 7 "2.2uF" H 3200 8600 50  0001 C CNN "Value"
-	1    3200 8600
+P 3150 8600
+F 0 "C14" V 3300 8550 50  0000 L CNN
+F 1 "2.2uF" V 3350 8500 50  0000 L CNN
+F 2 "Capacitor_SMD:C_0402_1005Metric" H 3188 8450 50  0001 C CNN
+F 3 "~" H 3150 8600 50  0001 C CNN
+F 4 "~" H 3150 8600 50  0001 C CNN "Datasheet"
+F 5 "Capacitor_SMD:C_0402_1005Metric" H 3150 8600 50  0001 C CNN "Footprint"
+F 6 "C14" H 3150 8600 50  0001 C CNN "Reference"
+F 7 "2.2uF" H 3150 8600 50  0001 C CNN "Value"
+	1    3150 8600
 	0    1    1    0
 $EndComp
-Connection ~ 3050 8600
-Connection ~ 3050 8300
-Wire Wire Line
-	3050 8700 3050 8600
-Wire Wire Line
-	3050 7700 3050 7800
-Text GLabel 3150 8000 2    50   Input ~ 0
+Connection ~ 3000 8600
+Connection ~ 3000 8300
+Wire Wire Line
+	3000 8700 3000 8600
+Wire Wire Line
+	3000 7700 3000 7800
+Text GLabel 3100 8000 2    50   Input ~ 0
 STM_SPI2_DRDY2
 Wire Wire Line
-	3050 8000 3150 8000
-Text GLabel 3150 7700 2    50   Input ~ 0
-SENSORS_3V3
-Wire Wire Line
-	3050 7700 3150 7700
-Text GLabel 3400 8450 2    50   Input ~ 0
-SENSORS_3V3
-NoConn ~ 1250 7800
-Wire Wire Line
-	1150 8400 1250 8400
-Wire Wire Line
-	1150 8100 1250 8100
-Wire Wire Line
-	1250 8200 1150 8200
-Wire Wire Line
-	1150 8300 1250 8300
+	3000 8000 3100 8000
+Wire Wire Line
+	3000 7700 3100 7700
+NoConn ~ 1200 7800
+Wire Wire Line
+	1150 8400 1200 8400
+Wire Wire Line
+	1150 8100 1200 8100
+Wire Wire Line
+	1200 8200 1150 8200
+Wire Wire Line
+	1150 8300 1200 8300
 Text GLabel 1150 8200 0    50   Input ~ 0
 STM_SPI2_SCK
@@
 Text Notes 550  7350 0    394  ~ 0
 ICM-42605
-Connection ~ 3050 7700
-Connection ~ 3050 8400
-Wire Wire Line
-	3050 8400 3050 8300
-Connection ~ 3050 8500
-Wire Wire Line
-	3050 8500 3050 8400
-Wire Wire Line
-	3050 8600 3050 8500
+Connection ~ 3000 7700
+Connection ~ 3000 8400
+Wire Wire Line
+	3000 8400 3000 8300
+Connection ~ 3000 8500
+Wire Wire Line
+	3000 8500 3000 8400
+Wire Wire Line
+	3000 8600 3000 8500
 $Comp
 L ICM-42605:ICM-42605 U7
 U 1 1 61BBA626
-P 2050 8200
-F 0 "U7" H 2050 8967 50  0000 C CNN
-F 1 "ICM-42605" H 2050 8876 50  0000 C CNN
-F 2 "ICM-42605:PQFN50P300X250X97-14N" H 2050 8200 50  0001 L BNN
-F 3 "" H 2050 8200 50  0001 L BNN
-F 4 "TDK Corporation" H 2050 8200 50  0001 L BNN "MANUFACTURER"
-F 5 "IPC 7351B" H 2050 8200 50  0001 L BNN "STANDARD"
-F 6 "0.4" H 2050 8200 50  0001 L BNN "PARTREV"
-F 7 "ICM-42605" H 2050 8200 50  0001 C CNN "Manufacturer_Part_Number"
-F 8 "ICM-42605:PQFN50P300X250X97-14N" H 2050 8200 50  0001 C CNN "Footprint"
-F 9 "U7" H 2050 8200 50  0001 C CNN "Reference"
-F 10 "ICM-42605" H 2050 8200 50  0001 C CNN "Value"
-	1    2050 8200
+P 2000 8200
+F 0 "U7" H 2000 8967 50  0000 C CNN
+F 1 "ICM-42605" H 2000 8876 50  0000 C CNN
+F 2 "ICM-42605:PQFN50P300X250X97-14N" H 2000 8200 50  0001 L BNN
+F 3 "" H 2000 8200 50  0001 L BNN
+F 4 "TDK Corporation" H 2000 8200 50  0001 L BNN "MANUFACTURER"
+F 5 "IPC 7351B" H 2000 8200 50  0001 L BNN "STANDARD"
+F 6 "0.4" H 2000 8200 50  0001 L BNN "PARTREV"
+F 7 "ICM-42605" H 2000 8200 50  0001 C CNN "Manufacturer_Part_Number"
+F 8 "ICM-42605:PQFN50P300X250X97-14N" H 2000 8200 50  0001 C CNN "Footprint"
+F 9 "U7" H 2000 8200 50  0001 C CNN "Reference"
+F 10 "ICM-42605" H 2000 8200 50  0001 C CNN "Value"
+	1    2000 8200
 	1    0    0    -1
 $EndComp
@@
 L power:GND #PWR0118
 U 1 1 61C507EE
-P 3050 8900
-F 0 "#PWR0118" H 3050 8650 50  0001 C CNN
-F 1 "GND" H 3055 8727 50  0000 C CNN
-F 2 "" H 3050 8900 50  0001 C CNN
-F 3 "" H 3050 8900 50  0001 C CNN
-	1    3050 8900
-	1    0    0    -1
-$EndComp
-Wire Wire Line
-	3050 8900 3050 8700
-Connection ~ 3050 8700
+P 3000 8900
+F 0 "#PWR0118" H 3000 8650 50  0001 C CNN
+F 1 "GND" H 3005 8727 50  0000 C CNN
+F 2 "" H 3000 8900 50  0001 C CNN
+F 3 "" H 3000 8900 50  0001 C CNN
+	1    3000 8900
+	1    0    0    -1
+$EndComp
+Wire Wire Line
+	3000 8900 3000 8700
+Connection ~ 3000 8700
 $Comp
 L power:GND #PWR0119
@@
 Wire Wire Line
 	2900 10450 2700 10450
-Wire Wire Line
-	3400 8450 3350 8450
-Connection ~ 3350 8450
-Wire Wire Line
-	3350 8450 3350 8600
-Text GLabel 2900 10150 2    50   Input ~ 0
-SENSORS_3V3
 Wire Wire Line
 	2700 10250 2700 10150
@@
 	2800 11050 2800 10150
 Connection ~ 2800 11050
-Wire Wire Line
-	2900 10150 2800 10150
 Connection ~ 2800 10150
 Wire Wire Line
@@
 Wire Wire Line
 	3000 11350 2800 11350
+Wire Wire Line
+	2900 10150 2800 10150
+Wire Wire Line
+	1200 4750 1250 4750
+Text Notes 500  5550 0    394  ~ 0
+BMM155
+Wire Wire Line
+	3300 8300 3300 8450
+Text GLabel 2500 5750 2    50   Input ~ 0
+SENSORS_3V3
+Text GLabel 3250 6250 2    50   Input ~ 0
+SENSORS_3V3
+Text GLabel 3000 3750 2    50   Input ~ 0
+SENSORS_3V3
+Text GLabel 1200 4750 0    50   Input ~ 0
+SENSORS_3V3
+Text GLabel 2900 1200 2    50   Input ~ 0
+SENSORS_3V3
+Text GLabel 3350 8450 2    50   Input ~ 0
+SENSORS_3V3
+Text GLabel 3100 7700 2    50   Input ~ 0
+SENSORS_3V3
+Text GLabel 2900 10150 2    50   Input ~ 0
+SENSORS_3V3
+Wire Wire Line
+	3300 8450 3350 8450
+Connection ~ 3300 8450
+Wire Wire Line
+	3300 8450 3300 8600
 $EndSCHEMATC
