File: ESP32.sch (KiCad schematic (older format))
At the start: 15 parts, among them IC1 LY68L6400SLIT, U10 ESP32-S2FH4, U11 W25Q128JVS, Y4 40MHz

Commit message: start migrating to kicad v6
Parts:
- U10: Footprint QFN40P700X700X90-57T400N -> ESP32-S2:QFN40P700X700X90-57T400N
Changed lines of the file:
@@
 F 6 "QFN-56" H 10950 4450 50  0001 L BNN "PACKAGE"
 F 7 "Espressif Systems" H 10950 4450 50  0001 L BNN "MANUFACTURER_NAME"
-F 8 "QFN40P700X700X90-57T400N" H 10950 4450 50  0001 C CNN "Footprint"
+F 8 "ESP32-S2:QFN40P700X700X90-57T400N" H 10950 4450 50  0001 C CNN "Footprint"
 F 9 "U10" H 10950 4450 50  0001 C CNN "Reference"
 F 10 "ESP32-S2FH4" H 10950 4450 50  0001 C CNN "Value"
