File: CopterCat_cm4.kicad_pcb (KiCad board)
At the start: 4 copper layers, 40 x 55 mm, 159 parts, among them IC1 LY68L6400SLIT, J2 Conn_01x08_Male, J3 Conn_01x08_Male, J4 Conn_01x08_Male, J5 5V, J6 USB_C_Receptacle_USB2.0, J7 USB_SWITCH, Q1 MMDT3906, Q2 DMP3013SFV, Q3 MUN5211DW1, Q4 AO3400A, Q5 AO3400A, Q6 2N7002K, Q7 FDN340P, Q8 DMP3013SFV, U1 STM32H753IIKx, U10 ESP32-S2FH4, U11 W25Q128JVS, U12 AMS1117-3.3, U13 74AHC1G04, U14 FSUSB42MUX, U15 TPD4E02B04DQA, U16 CAT24C256, U17 BMI088, U18 FSUSB42MUX, U19 USB2514B_Bi, U2 ICM-20602, U21 47579-0001, U3 BMP388, U4 FM25V02A-GTR, U5 BMM150, U6 Compute_Module_4_Connectors, U7 ICM-42605, U8 CP2104, U9 AMS1117-3.3, Y1 16MHz, Y2 32.768, Y3 24MHz, Y4 40MHz

Commit message: тестирование
Parts:
- removed F2, F3: BLM15BC241SN1D, Fuse:Fuse_0402_1005Metric
- added GND1: Conn_01x01_Male, TestPoint:TestPoint_Pad_D1.5mm, B.Cu at (240.8, 87.2)
- C17, C18, C3, C5, R11, R25, R26, R27: moved to B.Cu
- JP1, JP2: footprint Jumper:SolderJumper-2_P1.3mm_Open_TrianglePad1.0x1.5mm -> Jumper:SolderJumper-2_P1.3mm_Open_RoundedPad1.0x1.5mm
- LED1: value Conn_01x03_Male -> Conn_01x01_Male; footprint Connector_PinHeader_2.54mm:PinHeader_1x03_P2.54mm_Vertical -> TestPoint:TestPoint_Pad_D1.5mm
- moved C27 53.7 mm to (215.5, 97.7), turned to 180 degrees
- moved C24 52.8 mm to (239.4, 119.9)
- moved R19 29.7 mm to (229.4, 128.8), turned to 0 degrees
- moved R20 29.2 mm to (229.4, 127.8), turned to 180 degrees
- moved C5 21.2 mm to (218.8, 106.8), turned to 180 degrees
- moved C3 21.1 mm to (218.8, 105.8), turned to 180 degrees
- moved LED1 19.9 mm to (240.8, 87.2)
- moved C18 19.0 mm to (229.2, 127.5), turned to 0 degrees
- moved C17 17.6 mm to (229.2, 128.4), turned to 180 degrees
- moved C4 9.11 mm to (232.3, 123.8)
- moved U2 9.11 mm to (230.0, 124.4)
- moved U7 7.72 mm to (233.2, 120.7)
- moved C14 7.46 mm to (236.3, 120.7)
- moved C13 7.46 mm to (235.3, 120.7)
- moved R25 6.99 mm to (226.6, 110.5), turned to 0 degrees
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Connections:
- CAM0 pad MP: GND -> (no net)
- GPS1 pad MP: GND -> (no net)
- I2C1 pad MP: GND -> (no net)
- J5 pad 2: /Connectors/LED_V5 -> /Connectors/PWR_IN_CONN
- LASER1 pad MP: GND -> (no net)
- LED1 pad 1: /Connectors/LED_V5 -> /Connectors/RPI_GPIO21
- POWER1 pad MP: GND -> (no net)
- Q1 pad 1: /Connectors/LED_V5 -> /Connectors/PWR_IN_CONN
- Q2 pad 5: /Connectors/LED_V5 -> /Connectors/PWR_IN_CONN
- RC1 pad MP: GND -> (no net)
- TELEM1 pad MP: GND -> (no net)
- TELEM2 pad MP: GND -> (no net)
- U1 pad A10: STM_SDMMC2_D2 -> unconnected-(U1-PadA10)
- U1 pad A11: STM_SDMMC2_CMD -> unconnected-(U1-PadA11)
- U1 pad A13: /STM32/STM_SPI6.CS2 -> unconnected-(U1-PadA13)
- U1 pad A2: STM_TRACECLK -> unconnected-(U1-PadA2)
- U1 pad A3: /STM32/STM_UART8.TX -> unconnected-(U1-PadA3)
- U1 pad A4: /STM32/STM_UART8.RX -> unconnected-(U1-PadA4)
- U1 pad A6: /STM32/STM_OTG_HS_ULPI_D7 -> unconnected-(U1-PadA6)
- U1 pad A7: /STM32/STM_SPI6.MOSI -> unconnected-(U1-PadA7)
- U1 pad A8: /STM32/STM_SPI6.SCK -> unconnected-(U1-PadA8)
- U1 pad A9: STM_SDMMC2_D3 -> unconnected-(U1-PadA9)
- U1 pad B10: STM_VDD_5V_HIPOWER_NEN -> unconnected-(U1-PadB10)
- U1 pad B12: STM_CAN1_RX -> unconnected-(U1-PadB12)
- U1 pad B3: STM_NARMED -> unconnected-(U1-PadB3)
- U1 pad B7: STM_PG15 -> unconnected-(U1-PadB7)
- U1 pad C12: STM_CAN1_TX -> unconnected-(U1-PadC12)
- U1 pad D1: STM_VDD_3V3_SD_EN -> unconnected-(U1-PadD1)
- U1 pad D13: /STM32/STM_SPI4.CS1 -> unconnected-(U1-PadD13)
- U1 pad E12: /STM32/STM_UART4.TX -> unconnected-(U1-PadE12)
- U1 pad E13: /STM32/STM_UART4.RX -> unconnected-(U1-PadE13)
- U1 pad E2: /STM32/STM_I2C2.SDA -> unconnected-(U1-PadE2)
- U1 pad E3: /STM32/STM_SPI6.CS1 -> unconnected-(U1-PadE3)
- U1 pad E4: /STM32/STM_OTG_HS_ULPI_DIR -> unconnected-(U1-PadE4)
- U1 pad F15: /STM32/STM_I2C3.SCL -> unconnected-(U1-PadF15)
- U1 pad H14: STM_PG8 -> unconnected-(U1-PadH14)
- U1 pad H3: /STM32/STM_I2C2.SCL -> unconnected-(U1-PadH3)
- U1 pad J15: STM_PG6 -> unconnected-(U1-PadJ15)
- U1 pad J3: STM_PF4 -> unconnected-(U1-PadJ3)
- U1 pad K14: STM_VDD_5V_PERIPH_NEN -> unconnected-(U1-PadK14)
- U1 pad K15: STM_NPOWER_IN_C -> unconnected-(U1-PadK15)
- U1 pad K3: STM_SAFETY_SWITCH_IN -> unconnected-(U1-PadK3)
- U1 pad L1: /STM32/STM_SPI6.NRESET -> unconnected-(U1-PadL1)
- U1 pad L14: STM_PD15 -> unconnected-(U1-PadL14)
- U1 pad L15: STM_NPOWER_IN_B -> unconnected-(U1-PadL15)
- U1 pad L2: STM_BUZZER_1 -> unconnected-(U1-PadL2)
- U1 pad M12: /STM32/STM_I2C3.SDA -> unconnected-(U1-PadM12)
- U1 pad M2: /STM32/STM_OTG_HS_ULPI_STP -> unconnected-(U1-PadM2)
- U1 pad M3: STM_SDMMC2_CLK -> unconnected-(U1-PadM3)
- U1 pad M5: /STM32/STM_OTG_HS_ULPI_NXT -> unconnected-(U1-PadM5)
- U1 pad M7: STM_NPOWER_IN_A -> unconnected-(U1-PadM7)
- U1 pad N11: /STM32/STM_SPI4.MISO -> unconnected-(U1-PadN11)
- U1 pad N13: /STM32/STM_SPI6.DRDY2 -> unconnected-(U1-PadN13)
- U1 pad N14: /STM32/STM_SPI6.DRDY1 -> unconnected-(U1-PadN14)
- U1 pad N15: STM_NSAFETY_SWITCH_LED_OUT -> unconnected-(U1-PadN15)
- U1 pad N2: STM_CAP2 -> unconnected-(U1-PadN2)
- U1 pad N3: STM_V5_SCALED -> unconnected-(U1-PadN3)
- U1 pad N6: STM_5V_HIPOWER_NOC -> unconnected-(U1-PadN6)
- U1 pad P10: STM_CAP1 -> unconnected-(U1-PadP10)
- U1 pad P11: /STM32/STM_SPI4.MOSI -> unconnected-(U1-PadP11)
- U1 pad P12: /STM32/STM_OTG_HS_ULPI_D5 -> unconnected-(U1-PadP12)
- U1 pad P13: /STM32/STM_OTG_HS_ULPI_D6 -> unconnected-(U1-PadP13)
- U1 pad P2: STM_HEATER -> unconnected-(U1-PadP2)
- U1 pad P3: /STM32/STM_SPI6.MISO -> unconnected-(U1-PadP3)
- U1 pad P4: /STM32/STM_OTG_HS_ULPI_CK -> unconnected-(U1-PadP4)
- U1 pad P5: STM_MUX_CTRL1 -> unconnected-(U1-PadP5)
- U1 pad P6: STM_NFC_GPIO -> unconnected-(U1-PadP6)
- U1 pad P9: STM_SPIX_SYNC -> unconnected-(U1-PadP9)
- U1 pad R10: /STM32/STM_SPI4.SCK -> unconnected-(U1-PadR10)
- U1 pad R11: STM_5V_PERIPH_NOC -> unconnected-(U1-PadR11)
- U1 pad R12: /STM32/STM_OTG_HS_ULPI_D3 -> unconnected-(U1-PadR12)
- U1 pad R13: /STM32/STM_OTG_HS_ULPI_D4 -> unconnected-(U1-PadR13)
- U1 pad R14: STM_SDMMC2_D0 -> unconnected-(U1-PadR14)
- U1 pad R15: STM_SDMMC2_D1 -> unconnected-(U1-PadR15)
- U1 pad R2: /STM32/STM_OTG_HS_ULPI_D0 -> unconnected-(U1-PadR2)
- U1 pad R4: /STM32/STM_OTG_HS_ULPI_D2 -> unconnected-(U1-PadR4)
- U1 pad R5: /STM32/STM_OTG_HS_ULPI_D1 -> unconnected-(U1-PadR5)
- U1 pad R8: STM_MUX_CTRL2 -> unconnected-(U1-PadR8)
- U10 pad 1: Net-(F3-Pad2) -> /ESP32/ESP_3V3
- U10 pad 20: Net-(F2-Pad2) -> /ESP32/ESP_3V3
- U10 pad 27: Net-(F2-Pad2) -> /ESP32/ESP_3V3
- U10 pad 3: Net-(F3-Pad2) -> /ESP32/ESP_3V3
- U10 pad 4: Net-(F3-Pad2) -> /ESP32/ESP_3V3
- U10 pad 45: Net-(F3-Pad2) -> /ESP32/ESP_3V3
- U10 pad 51: Net-(F3-Pad2) -> /ESP32/ESP_3V3
- U10 pad 54: Net-(F3-Pad2) -> /ESP32/ESP_3V3
Routing:
- net /STM32/SENSORS_3V3: track 75.8 -> 0.00 mm, vias 11 -> 0
- net /Connectors/STM_ESC.CH8: track 71.6 -> 0.46 mm
- net /STM32/STM_USB.VBUS: track 83.9 -> 13.1 mm, vias 6 -> 3
- net /Power/3V3_GROUP1: track 124.3 -> 55.2 mm, vias 20 -> 11
- net /Connectors/STM_ESC.CH7: track 69.2 -> 0.44 mm
- net /RPi_CM4/RPI_USB.ID: track 68.5 -> 0.00 mm, vias 3 -> 0
- net /Connectors/STM_ESC.CH2: track 66.1 -> 0.46 mm
- net /Connectors/STM_ESC.CH6: track 61.9 -> 0.46 mm
- net /Connectors/STM_ESC.CH4: track 60.6 -> 0.46 mm
- net /Connectors/STM_ESC.CH5: track 59.6 -> 0.55 mm
- net /Connectors/RPI_CAM_GPIO: track 56.5 -> 0.00 mm, vias 2 -> 0
- net /Connectors/STM_ESC.CH3: track 54.1 -> 0.46 mm, vias 2 -> 1
- net /Connectors/STM_ESC.CH1: track 53.7 -> 0.47 mm
- net /Connectors/USB_BOARD.DP: track 51.6 -> 2.88 mm, vias 3 -> 0
- net /Connectors/RPI_I2C1.SCL: track 47.7 -> 0.00 mm, vias 3 -> 0
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- added copper zone on In1.Cu, net GND
- added copper zone on In2.Cu, net GND

Commit message: second version
Parts:
- C10, JP1, R23, R24, R28, R7: moved to B.Cu
- moved C10 15.0 mm to (222.3, 111.0), turned to 90 degrees
- moved R28 14.3 mm to (223.2, 111.0)
- moved JP1 9.81 mm to (226.1, 107.5), turned to 0 degrees
- moved R17 9.09 mm to (232.2, 93.9)
- moved R23 8.80 mm to (225.1, 109.2), turned to 0 degrees
- moved C27 7.90 mm to (220.8, 91.8)
- moved R33 7.53 mm to (231.9, 110.8), turned to 0 degrees
- moved R32 6.61 mm to (231.9, 109.9), turned to 180 degrees
- moved R24 6.55 mm to (228.0, 107.5), turned to -90 degrees
- moved R7 6.03 mm to (227.0, 109.2), turned to 0 degrees
- moved R31 5.86 mm to (231.9, 109.0), turned to 0 degrees
- moved C2 4.58 mm to (226.3, 118.3), turned to 90 degrees
- moved D1 4.25 mm to (234.3, 109.7), turned to -90 degrees
- moved C21 3.17 mm to (231.7, 102.1), turned to 90 degrees
- moved C1 2.95 mm to (221.4, 118.3)
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Connections:
- U1 pad D10: /ESP32/ESP_UART1.RTS -> unconnected-(U1-PadD10)
- U1 pad D11: /ESP32/ESP_UART1.CTS -> unconnected-(U1-PadD11)
- U1 pad F14: /Connectors/STM_UART5.CTS -> unconnected-(U1-PadF14)
- U1 pad G14: /Connectors/STM_UART5.RTS -> unconnected-(U1-PadG14)
- U1 pad L3: /Connectors/STM_UART7.RTS -> unconnected-(U1-PadL3)
- U1 pad R9: /Connectors/STM_UART7.CTS -> unconnected-(U1-PadR9)
Routing:
- net /STM32/STM_USB.VBUS: track 13.1 -> 80.1 mm, vias 3 -> 6
- net /Connectors/STM_ESC.CH1: track 0.47 -> 50.6 mm
- net /Connectors/STM_ESC.CH2: track 0.46 -> 49.2 mm
- net /Connectors/STM_ESC.CH7: track 0.44 -> 49.1 mm
- net /Connectors/STM_ESC.CH3: track 0.46 -> 46.8 mm
- net /Connectors/STM_ESC.CH4: track 0.46 -> 45.6 mm
- net /Connectors/STM_ESC.CH8: track 0.46 -> 44.0 mm
- net /Connectors/STM_ESC.CH5: track 0.55 -> 43.1 mm
- net /Connectors/STM_ESC.CH6: track 0.46 -> 42.5 mm
- net /Connectors/USB_BOARD.DN: track 2.93 -> 43.1 mm, vias 0 -> 2
- net /Connectors/USB_BOARD.DP: track 2.88 -> 41.3 mm, vias 0 -> 2
- net /RPi_CM4/RPI_USB.ID: track 0.00 -> 35.5 mm, vias 0 -> 4
- net /STM32/STM_USB.DP: track 0.00 -> 31.8 mm, vias 0 -> 2
- net /STM32/STM_USB.DN: track 0.00 -> 30.0 mm, vias 0 -> 2
- net /RPi_CM4/RPI_USB.DN: track 0.00 -> 29.2 mm, vias 0 -> 2
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