File: BMM150.kicad_sch (KiCad schematic)
At the start: 4 parts, among them U5 BMM150

Commit message: Little fix
Parts:
- C36, C37: Manufacturer_Part_Number (none) -> CL05B104KB54PNC
- R41: Manufacturer_Part_Number (none) -> 0402WGF1002TCE
Changed lines of the file:
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@@
+      (effects (font (size 1.27 1.27)) hide)
+    )
+    (property "Manufacturer_Part_Number" "CL05B104KB54PNC" (id 4) (at 120.65 67.31 0)
       (effects (font (size 1.27 1.27)) hide)
     )
@@
     )
     (property "Datasheet" "~" (id 3) (at 104.14 63.5 0)
+      (effects (font (size 1.27 1.27)) hide)
+    )
+    (property "Manufacturer_Part_Number" "0402WGF1002TCE" (id 4) (at 104.14 63.5 0)
       (effects (font (size 1.27 1.27)) hide)
     )
@@
       (effects (font (size 1.27 1.27)) hide)
     )
+    (property "Manufacturer_Part_Number" "CL05B104KB54PNC" (id 4) (at 109.22 67.31 0)
+      (effects (font (size 1.27 1.27)) hide)
+    )

Commit message: First order
Parts:
- C36, C37: Manufacturer_Part_Number CL05B104KB54PNC -> C1005X7R1H104KT000S
- R41: Manufacturer_Part_Number 0402WGF1002TCE -> RNCF0402BTE10K0
Changed lines of the file:
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@@
       (effects (font (size 1.27 1.27)) hide)
     )
-    (property "Manufacturer_Part_Number" "CL05B104KB54PNC" (id 4) (at 120.65 67.31 0)
+    (property "Manufacturer_Part_Number" "C1005X7R1H104KT000S" (id 4) (at 120.65 67.31 0)
       (effects (font (size 1.27 1.27)) hide)
     )
@@
       (effects (font (size 1.27 1.27)) hide)
     )
-    (property "Manufacturer_Part_Number" "0402WGF1002TCE" (id 4) (at 104.14 63.5 0)
+    (property "Manufacturer_Part_Number" "RNCF0402BTE10K0" (id 4) (at 104.14 63.5 0)
       (effects (font (size 1.27 1.27)) hide)
     )
@@
       (effects (font (size 1.27 1.27)) hide)
     )
-    (property "Manufacturer_Part_Number" "CL05B104KB54PNC" (id 4) (at 109.22 67.31 0)
+    (property "Manufacturer_Part_Number" "C1005X7R1H104KT000S" (id 4) (at 109.22 67.31 0)
       (effects (font (size 1.27 1.27)) hide)
     )
