File: BMP388.kicad_sch (KiCad schematic)
At the start: 3 parts, among them U3 BMP388

Commit message: Little fix
Parts:
- C6, C7: Manufacturer_Part_Number (none) -> CL05B104KB54PNC
Changed lines of the file:
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@@
+      (effects (font (size 1.27 1.27)) hide)
+    )
+    (property "Manufacturer_Part_Number" "CL05B104KB54PNC" (id 4) (at 124.46 68.58 0)
       (effects (font (size 1.27 1.27)) hide)
     )
@@
       (effects (font (size 1.27 1.27)) hide)
     )
+    (property "Manufacturer_Part_Number" "CL05B104KB54PNC" (id 4) (at 113.03 68.58 0)
+      (effects (font (size 1.27 1.27)) hide)
+    )

Commit message: First order
Parts:
- C6, C7: Manufacturer_Part_Number CL05B104KB54PNC -> C1005X7R1H104KT000S
Changed lines of the file:
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@@
       (effects (font (size 1.27 1.27)) hide)
     )
-    (property "Manufacturer_Part_Number" "CL05B104KB54PNC" (id 4) (at 124.46 68.58 0)
+    (property "Manufacturer_Part_Number" "C1005X7R1H104KT000S" (id 4) (at 124.46 68.58 0)
       (effects (font (size 1.27 1.27)) hide)
     )
@@
       (effects (font (size 1.27 1.27)) hide)
     )
-    (property "Manufacturer_Part_Number" "CL05B104KB54PNC" (id 4) (at 113.03 68.58 0)
+    (property "Manufacturer_Part_Number" "C1005X7R1H104KT000S" (id 4) (at 113.03 68.58 0)
       (effects (font (size 1.27 1.27)) hide)
     )
