File: ESP32.kicad_sch (KiCad schematic)
At the start: 24 parts, among them IC1 LY68L6400SLIT, U10 ESP32-S2FH4, U11 W25Q128JVS, Y4 40MHz

Commit message: плата практически готова
Parts:
- added C38: 10uF, Capacitor_Tantalum_SMD:CP_EIA-3216-18_Kemet-A, symbol Device:C_Polarized
- ANT1: footprint ANT_ANT016008LCS2442MA2 -> ANT016008LCS2442MA2:ANT_ANT016008LCS2442MA2
- Q3: renamed from Q?; Manufacturer_Part_Number (none) -> MUN5211DW1T1G
- gave numbers to parts that had none: 5
Connections:
- net ESP_3V3: now also C38.1
- net GND: now also C38.2
Changed lines of the file:
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@@
   (junction (at 100.33 34.29) (diameter 0) (color 0 0 0 0)
+  )
+  (junction (at 149.86 22.86) (diameter 0) (color 0 0 0 0)
   )
   (junction (at 138.43 30.48) (diameter 0) (color 0 0 0 0)
@@
     (stroke (width 0) (type default) (color 0 0 0 0))
   )
+  (wire (pts (xy 138.43 30.48) (xy 149.86 30.48))
+    (stroke (width 0) (type default) (color 0 0 0 0))
+  )
   (polyline (pts (xy 199.39 130.81) (xy 12.7 130.81))
     (stroke (width 0) (type default) (color 0 0 0 0))
@@
     (stroke (width 0) (type default) (color 0 0 0 0))
   )
-  (wire (pts (xy 147.32 22.86) (xy 138.43 22.86))
+  (wire (pts (xy 154.94 22.86) (xy 149.86 22.86))
     (stroke (width 0) (type default) (color 0 0 0 0))
   )
@@
   )
   (wire (pts (xy 110.49 214.63) (xy 110.49 212.09))
+    (stroke (width 0) (type default) (color 0 0 0 0))
+  )
+  (wire (pts (xy 149.86 22.86) (xy 138.43 22.86))
     (stroke (width 0) (type default) (color 0 0 0 0))
   )
@@
     (effects (font (size 1.27 1.27)) (justify right))
   )
-  (hierarchical_label "ESP_3V3" (shape input) (at 147.32 22.86 0)
+  (hierarchical_label "ESP_3V3" (shape input) (at 154.94 22.86 0)
     (effects (font (size 1.27 1.27)) (justify left))
   )
@@
   (symbol (lib_id "Transistor_BJT:MUN5211DW1") (at 109.22 219.71 0) (unit 2)
     (in_bom yes) (on_board yes) (fields_autoplaced)
-    (property "Reference" "Q?" (id 0) (at 112.8014 218.9793 0)
+    (property "Reference" "Q3" (id 0) (at 112.8014 218.9793 0)
       (effects (font (size 1.27 1.27)) (justify left))
     )
@@
       (effects (font (size 1.27 1.27)) hide)
     )
+    (property "Manufacturer_Part_Number" "MUN5211DW1T1G" (id 4) (at 109.22 219.71 0)
+      (effects (font (size 1.27 1.27)) hide)
+    )
     (pin "1")
     (pin "2")
@@
       (effects (font (size 1.27 1.27)) (justify left))
     )
-    (property "Footprint" "ANT_ANT016008LCS2442MA2" (id 2) (at 182.88 44.45 0)
+    (property "Footprint" "ANT016008LCS2442MA2:ANT_ANT016008LCS2442MA2" (id 2) (at 182.88 44.45 0)
       (effects (font (size 1.27 1.27)) (justify left bottom) hide)
     )
@@
   (symbol (lib_id "Interface_USB:CP2104") (at 60.96 180.34 0) (unit 1)
     (in_bom yes) (on_board yes) (fields_autoplaced)
-    (property "Reference" "U?" (id 0) (at 62.9794 207.8895 0)
+    (property "Reference" "U8" (id 0) (at 62.9794 207.8895 0)
       (effects (font (size 1.27 1.27)) (justify left))
     )
@@
   (symbol (lib_id "Device:R") (at 58.42 93.98 90) (unit 1)
     (in_bom yes) (on_board yes)
-    (property "Reference" "R?" (id 0) (at 58.42 99.2378 90))
+    (property "Reference" "R42" (id 0) (at 58.42 99.2378 90))
     (property "Value" "1K" (id 1) (at 58.42 96.9264 90))
     (property "Footprint" "Resistor_SMD:R_0402_1005Metric" (id 2) (at 58.42 95.758 90)
@@
     (pin "2")
   )
+  (symbol (lib_id "Device:C_Polarized") (at 149.86 26.67 0) (unit 1)
+    (in_bom yes) (on_board yes) (fields_autoplaced)
+    (property "Reference" "C38" (id 0) (at 152.781 24.8725 0)
+      (effects (font (size 1.27 1.27)) (justify left))
+    )
+    (property "Value" "10uF" (id 1) (at 152.781 27.6476 0)
+      (effects (font (size 1.27 1.27)) (justify left))
+    )
+    (property "Footprint" "Capacitor_Tantalum_SMD:CP_EIA-3216-18_Kemet-A" (id 2) (at 150.8252 30.48 0)
+      (effects (font (size 1.27 1.27)) hide)
+    )
+    (property "Datasheet" "~" (id 3) (at 149.86 26.67 0)
+      (effects (font (size 1.27 1.27)) hide)
+    )
+    (property "Manufacturer_Part_Number" "CL31A226KAHNNNE" (id 4) (at 149.86 26.67 0)
+      (effects (font (size 1.27 1.27)) hide)
+    )
+    (pin "1")
+    (pin "2")
+  )
   (symbol (lib_id "Device:C") (at 130.81 200.66 0) (unit 1)
     (in_bom yes) (on_board yes)
-    (property "Reference" "C?" (id 0) (at 133.731 199.4916 0)
+    (property "Reference" "C19" (id 0) (at 133.731 199.4916 0)
       (effects (font (size 1.27 1.27)) (justify left))
     )
@@
   (symbol (lib_id "Device:R") (at 58.42 91.44 270) (unit 1)
     (in_bom yes) (on_board yes)
-    (property "Reference" "R?" (id 0) (at 58.42 86.1822 90))
+    (property "Reference" "R14" (id 0) (at 58.42 86.1822 90))
     (property "Value" "1K" (id 1) (at 58.42 88.4936 90))
     (property "Footprint" "Resistor_SMD:R_0402_1005Metric" (id 2) (at 58.42 89.662 90)
@@
   (symbol (lib_id "power:GND") (at 130.81 205.74 0) (unit 1)
     (in_bom yes) (on_board yes)
-    (property "Reference" "#PWR?" (id 0) (at 130.81 212.09 0)
+    (property "Reference" "#PWR0123" (id 0) (at 130.81 212.09 0)
       (effects (font (size 1.27 1.27)) hide)
     )
@@
   (symbol (lib_id "Transistor_BJT:MUN5211DW1") (at 109.22 203.2 0) (unit 1)
     (in_bom yes) (on_board yes) (fields_autoplaced)
-    (property "Reference" "Q?" (id 0) (at 112.8014 202.4693 0)
+    (property "Reference" "Q3" (id 0) (at 112.8014 202.4693 0)
       (effects (font (size 1.27 1.27)) (justify left))
     )
@@
   (symbol (lib_id "power:GND") (at 60.96 210.82 0) (unit 1)
     (in_bom yes) (on_board yes)
-    (property "Reference" "#PWR?" (id 0) (at 60.96 217.17 0)
-      (effects (font (size 1.27 1.27)) hide)
-    )
+    (property "Reference" "#PWR0101" (id 0) (at 60.96 217.17 0)
+      (effects (font (size 1.27 1.27)) hide)
+    )

Commit message: продам гараж
Parts:
- removed Y4: 40MHz, Crystal:Crystal_SMD_2016-4Pin_2.0x1.6mm, symbol Device:Crystal_GND2
- added Y4: 40MHz, Crystal:Crystal_SMD_2016-4Pin_2.0x1.6mm, symbol Device:Crystal_GND24
Connections:
- net ESP_UART1.RX: now also U10.15 (IO10); no longer U10.50 (IO45)
- net ESP_UART1.TX: now also U10.16 (IO11); no longer U10.55 (IO46)
- net GND: now also Y4.2, Y4.4
- net at C31.1, U10.52 (XTAL_N): now also Y4.3
- net at C30.2, U10.53 (XTAL_P): now also Y4.1
Other:
- moved on the sheet: L1
Changed lines of the file:
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@@
   (junction (at 87.63 34.29) (diameter 0) (color 0 0 0 0)
+  )
+  (junction (at 25.4 69.85) (diameter 0) (color 0 0 0 0)
   )
   (junction (at 102.87 34.29) (diameter 0) (color 0 0 0 0)
@@
   (no_connect (at 73.66 172.72))
   (no_connect (at 73.66 175.26))
-  (bus_entry (at 148.59 104.14) (size -2.54 2.54)
+  (bus_entry (at 148.59 68.58) (size -2.54 2.54)
     (stroke (width 0) (type default) (color 0 0 0 0))
   )
@@
     (stroke (width 0) (type default) (color 0 0 0 0))
   )
-  (bus_entry (at 148.59 106.68) (size -2.54 2.54)
-    (stroke (width 0) (type default) (color 0 0 0 0))
-  )
-  (bus (pts (xy 148.59 106.68) (xy 148.59 104.14))
+  (bus_entry (at 148.59 71.12) (size -2.54 2.54)
+    (stroke (width 0) (type default) (color 0 0 0 0))
+  )
+  (bus (pts (xy 148.59 71.12) (xy 148.59 68.58))
     (stroke (width 0) (type default) (color 0 0 0 0))
   )
@@
     (stroke (width 0) (type default) (color 0 0 0 0))
   )
-  (polyline (pts (xy 129.54 110.49) (xy 143.51 110.49))
+  (polyline (pts (xy 129.54 74.93) (xy 143.51 74.93))
     (stroke (width 0) (type default) (color 0 0 0 0))
   )
@@
     (stroke (width 0) (type default) (color 0 0 0 0))
   )
+  (wire (pts (xy 25.4 55.88) (xy 25.4 69.85))
+    (stroke (width 0) (type default) (color 0 0 0 0))
+  )
   (wire (pts (xy 34.29 172.72) (xy 48.26 172.72))
     (stroke (width 0) (type default) (color 0 0 0 0))
   )
+  (wire (pts (xy 25.4 69.85) (xy 30.48 69.85))
+    (stroke (width 0) (type default) (color 0 0 0 0))
+  )
   (wire (pts (xy 63.5 66.04) (xy 66.04 66.04))
     (stroke (width 0) (type default) (color 0 0 0 0))
@@
     (stroke (width 0) (type default) (color 0 0 0 0))
   )
-  (wire (pts (xy 127 109.22) (xy 146.05 109.22))
+  (wire (pts (xy 127 73.66) (xy 146.05 73.66))
     (stroke (width 0) (type default) (color 0 0 0 0))
   )
@@
     (stroke (width 0) (type default) (color 0 0 0 0))
   )
-  (wire (pts (xy 140.97 57.15) (xy 140.97 58.42))
+  (wire (pts (xy 140.97 55.88) (xy 140.97 57.15))
     (stroke (width 0) (type default) (color 0 0 0 0))
   )
@@
     (stroke (width 0) (type default) (color 0 0 0 0))
   )
-  (bus (pts (xy 148.59 104.14) (xy 148.59 102.87))
+  (bus (pts (xy 148.59 68.58) (xy 148.59 67.31))
     (stroke (width 0) (type default) (color 0 0 0 0))
   )
@@
     (stroke (width 0) (type default) (color 0 0 0 0))
   )
-  (bus (pts (xy 148.59 109.22) (xy 148.59 106.68))
+  (bus (pts (xy 148.59 73.66) (xy 148.59 71.12))
     (stroke (width 0) (type default) (color 0 0 0 0))
   )
@@
     (stroke (width 0) (type default) (color 0 0 0 0))
   )
+  (wire (pts (xy 30.48 57.15) (xy 30.48 55.88))
+    (stroke (width 0) (type default) (color 0 0 0 0))
+  )
   (wire (pts (xy 76.2 160.02) (xy 73.66 160.02))
     (stroke (width 0) (type default) (color 0 0 0 0))
@@
     (stroke (width 0) (type default) (color 0 0 0 0))
   )
-  (wire (pts (xy 127 106.68) (xy 146.05 106.68))
+  (wire (pts (xy 127 71.12) (xy 146.05 71.12))
     (stroke (width 0) (type default) (color 0 0 0 0))
   )
@@
     (stroke (width 0) (type default) (color 0 0 0 0))
   )
+  (wire (pts (xy 30.48 55.88) (xy 25.4 55.88))
+    (stroke (width 0) (type default) (color 0 0 0 0))
+  )
   (wire (pts (xy 127 30.48) (xy 138.43 30.48))
     (stroke (width 0) (type default) (color 0 0 0 0))
@@
     (stroke (width 0) (type default) (color 0 0 0 0))
   )
-  (wire (pts (xy 140.97 41.91) (xy 140.97 44.45))
+  (wire (pts (xy 140.97 41.91) (xy 140.97 43.18))
     (stroke (width 0) (type default) (color 0 0 0 0))
   )
@@
     (stroke (width 0) (type default) (color 0 0 0 0))
   )
-  (polyline (pts (xy 129.54 99.06) (xy 129.54 110.49))
+  (polyline (pts (xy 129.54 63.5) (xy 129.54 74.93))
     (stroke (width 0) (type default) (color 0 0 0 0))
   )
@@
     (stroke (width 0) (type default) (color 0 0 0 0))
   )
-  (bus (pts (xy 148.59 102.87) (xy 149.86 102.87))
+  (bus (pts (xy 148.59 67.31) (xy 149.86 67.31))
     (stroke (width 0) (type default) (color 0 0 0 0))
   )
@@
     (stroke (width 0) (type default) (color 0 0 0 0))
   )
-  (wire (pts (xy 21.59 69.85) (xy 30.48 69.85))
-    (stroke (width 0) (type default) (color 0 0 0 0))
-  )
-  (polyline (pts (xy 129.54 99.06) (xy 143.51 99.06))
+  (wire (pts (xy 21.59 69.85) (xy 25.4 69.85))
+    (stroke (width 0) (type default) (color 0 0 0 0))
+  )
+  (polyline (pts (xy 129.54 63.5) (xy 143.51 63.5))
     (stroke (width 0) (type default) (color 0 0 0 0))
   )
@@
     (stroke (width 0) (type default) (color 0 0 0 0))
   )
-  (polyline (pts (xy 143.51 110.49) (xy 143.51 99.06))
+  (polyline (pts (xy 143.51 74.93) (xy 143.51 63.5))
     (stroke (width 0) (type default) (color 0 0 0 0))
   )
@@
     (effects (font (size 10.0076 10.0076)) (justify left bottom))
   )
-  (text "SOFT \nSWAP\n" (at 130.81 104.14 0)
+  (text "SOFT \nSWAP\n" (at 130.81 68.58 0)
     (effects (font (size 1.27 1.27)) (justify left bottom))
   )
@@
     (effects (font (size 1.27 1.27)) (justify left bottom))
   )
-  (label "ESP_UART1.RX" (at 129.54 106.68 0)
-    (effects (font (size 1.27 1.27)) (justify left bottom))
-  )
-  (label "ESP_UART1.TX" (at 129.54 109.22 0)
+  (label "ESP_UART1.RX" (at 129.54 71.12 0)
+    (effects (font (size 1.27 1.27)) (justify left bottom))
+  )
+  (label "ESP_UART1.TX" (at 129.54 73.66 0)
     (effects (font (size 1.27 1.27)) (justify left bottom))
   )
@@
     (effects (font (size 1.27 1.27)) (justify right bottom))
   )
-  (hierarchical_label "ESP_UART1{UART}" (shape input) (at 149.86 102.87 0)
+  (hierarchical_label "ESP_UART1{UART}" (shape input) (at 149.86 67.31 0)
     (effects (font (size 1.27 1.27)) (justify left))
   )
@@
     (pin "2")
   )
-  (symbol (lib_id "Device:Crystal_GND2") (at 30.48 62.23 0) (unit 1)
-    (in_bom yes) (on_board yes)
-    (property "Reference" "Y4" (id 0) (at 30.48 55.4228 0))
-    (property "Value" "40MHz" (id 1) (at 30.48 57.7342 0))
-    (property "Footprint" "Crystal:Crystal_SMD_2016-4Pin_2.0x1.6mm" (id 2) (at 30.48 62.23 0)
-      (effects (font (size 1.27 1.27)) hide)
-    )
-    (property "Datasheet" "~" (id 3) (at 30.48 62.23 0)
-      (effects (font (size 1.27 1.27)) hide)
-    )
-    (property "Manufacturer_Part_Number" "OT201640MJBA4SL" (id 4) (at 30.48 62.23 0)
-      (effects (font (size 1.27 1.27)) hide)
-    )
-    (pin "1")
-    (pin "2")
-    (pin "3")
-  )
   (symbol (lib_id "Device:C") (at 21.59 66.04 180) (unit 1)
     (in_bom yes) (on_board yes)
@@
     )
     (pin "1")
+  )
+  (symbol (lib_id "Device:Crystal_GND24") (at 30.48 62.23 0) (unit 1)
+    (in_bom yes) (on_board yes)
+    (property "Reference" "Y4" (id 0) (at 30.48 50.5649 0))
+    (property "Value" "40MHz" (id 1) (at 30.48 53.34 0))
+    (property "Footprint" "Crystal:Crystal_SMD_2016-4Pin_2.0x1.6mm" (id 2) (at 30.48 62.23 0)
+      (effects (font (size 1.27 1.27)) hide)
+    )
+    (property "Datasheet" "~" (id 3) (at 30.48 62.23 0)
+      (effects (font (size 1.27 1.27)) hide)
+    )
+    (property "Manufacturer_Part_Number" "OT201640MJBA4SL" (id 4) (at 30.48 62.23 0)
+      (effects (font (size 1.27 1.27)) hide)
+    )
+    (pin "1")
+    (pin "2")
+    (pin "3")
+    (pin "4")
   )
   (symbol (lib_id "Transistor_BJT:MUN5211DW1") (at 109.22 219.71 0) (unit 2)
@@
     (pin "2")
   )
-  (symbol (lib_id "pspice:INDUCTOR") (at 140.97 50.8 270) (unit 1)
+  (symbol (lib_id "pspice:INDUCTOR") (at 140.97 49.53 270) (unit 1)
     (in_bom yes) (on_board yes) (fields_autoplaced)
-    (property "Reference" "L1" (id 0) (at 142.875 49.8915 90)
-      (effects (font (size 1.27 1.27)) (justify left))
-    )
-    (property "Value" "3nH" (id 1) (at 142.875 52.6666 90)
-      (effects (font (size 1.27 1.27)) (justify left))
-    )
-    (property "Footprint" "Inductor_SMD:L_0402_1005Metric" (id 2) (at 140.97 50.8 0)
-      (effects (font (size 1.27 1.27)) hide)
-    )
-    (property "Datasheet" "~" (id 3) (at 140.97 50.8 0)
-      (effects (font (size 1.27 1.27)) hide)
-    )
-    (property "Manufacturer_Part_Number" "SDCL1005C2N0STDF" (id 4) (at 140.97 50.8 0)
-      (effects (font (size 1.27 1.27)) hide)
-    )
-    (pin "1")
-    (pin "2")
-  )
-  (symbol (lib_id "power:GND") (at 140.97 58.42 0) (unit 1)
-    (in_bom yes) (on_board yes)
-    (property "Reference" "#PWR0104" (id 0) (at 140.97 64.77 0)
-      (effects (font (size 1.27 1.27)) hide)
-    )
-    (property "Value" "GND" (id 1) (at 141.097 62.8142 0))
-    (property "Footprint" "" (id 2) (at 140.97 58.42 0)
-      (effects (font (size 1.27 1.27)) hide)
-    )
-    (property "Datasheet" "" (id 3) (at 140.97 58.42 0)
-      (effects (font (size 1.27 1.27)) hide)
-    )
+    (property "Reference" "L1" (id 0) (at 142.875 48.6215 90)
+      (effects (font (size 1.27 1.27)) (justify left))
+    )
+    (property "Value" "3nH" (id 1) (at 142.875 51.3966 90)
+      (effects (font (size 1.27 1.27)) (justify left))
+    )
+    (property "Footprint" "Inductor_SMD:L_0402_1005Metric" (id 2) (at 140.97 49.53 0)
+      (effects (font (size 1.27 1.27)) hide)
+    )
+    (property "Datasheet" "~" (id 3) (at 140.97 49.53 0)
+      (effects (font (size 1.27 1.27)) hide)
+    )
+    (property "Manufacturer_Part_Number" "SDCL1005C2N0STDF" (id 4) (at 140.97 49.53 0)
+      (effects (font (size 1.27 1.27)) hide)
+    )
+    (pin "1")
+    (pin "2")
+  )
+  (symbol (lib_id "power:GND") (at 140.97 57.15 0) (unit 1)
+    (in_bom yes) (on_board yes)
+    (property "Reference" "#PWR0104" (id 0) (at 140.97 63.5 0)
+      (effects (font (size 1.27 1.27)) hide)
+    )
+    (property "Value" "GND" (id 1) (at 141.097 61.5442 0))
+    (property "Footprint" "" (id 2) (at 140.97 57.15 0)
+      (effects (font (size 1.27 1.27)) hide)
+    )
+    (property "Datasheet" "" (id 3) (at 140.97 57.15 0)
+      (effects (font (size 1.27 1.27)) hide)
+    )

Commit message: )
Connections:
- no-connect marks 12 -> 41
Changed lines of the file:
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@@
   (junction (at 220.98 90.17) (diameter 0) (color 0 0 0 0)
   )
+  (no_connect (at 127 101.6))
+  (no_connect (at 127 99.06))
+  (no_connect (at 127 96.52))
+  (no_connect (at 127 93.98))
+  (no_connect (at 127 91.44))
+  (no_connect (at 127 114.3))
+  (no_connect (at 127 111.76))
+  (no_connect (at 127 109.22))
+  (no_connect (at 127 106.68))
+  (no_connect (at 127 104.14))
+  (no_connect (at 127 88.9))
+  (no_connect (at 127 63.5))
+  (no_connect (at 127 60.96))
+  (no_connect (at 127 48.26))
+  (no_connect (at 127 50.8))
+  (no_connect (at 127 53.34))
+  (no_connect (at 127 55.88))
+  (no_connect (at 127 58.42))
+  (no_connect (at 127 86.36))
+  (no_connect (at 127 83.82))
+  (no_connect (at 127 81.28))
+  (no_connect (at 127 78.74))
+  (no_connect (at 127 76.2))
+  (no_connect (at 127 66.04))
+  (no_connect (at 127 68.58))
+  (no_connect (at 66.04 80.01))
+  (no_connect (at 66.04 87.63))
+  (no_connect (at 66.04 85.09))
+  (no_connect (at 66.04 82.55))
   (no_connect (at 73.66 187.96))
   (no_connect (at 73.66 182.88))
