File: ICM20602.kicad_sch (KiCad schematic)
At the start: 4 parts, among them U2 ICM-20602

Commit message: Little fix
Parts:
- C3: Manufacturer_Part_Number (none) -> CL05A225MQ5NSNC
- C4, C5: Manufacturer_Part_Number (none) -> CL05B104KB54PNC
Changed lines of the file:
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@@
+      (effects (font (size 1.27 1.27)) hide)
+    )
+    (property "Manufacturer_Part_Number" "CL05B104KB54PNC" (id 4) (at 111.76 76.2 0)
       (effects (font (size 1.27 1.27)) hide)
     )
@@
     )
     (property "Datasheet" "~" (id 3) (at 119.38 52.07 0)
+      (effects (font (size 1.27 1.27)) hide)
+    )
+    (property "Manufacturer_Part_Number" "CL05B104KB54PNC" (id 4) (at 119.38 52.07 0)
       (effects (font (size 1.27 1.27)) hide)
     )
@@
       (effects (font (size 1.27 1.27)) hide)
     )
+    (property "Manufacturer_Part_Number" "CL05A225MQ5NSNC" (id 4) (at 107.95 52.07 0)
+      (effects (font (size 1.27 1.27)) hide)
+    )

Commit message: First order
Parts:
- C3: Manufacturer_Part_Number CL05A225MQ5NSNC -> ZRB157R61C225KE11D
- C4, C5: Manufacturer_Part_Number CL05B104KB54PNC -> C1005X7R1H104KT000S
Changed lines of the file:
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@@
       (effects (font (size 1.27 1.27)) hide)
     )
-    (property "Manufacturer_Part_Number" "CL05B104KB54PNC" (id 4) (at 111.76 76.2 0)
+    (property "Manufacturer_Part_Number" "C1005X7R1H104KT000S" (id 4) (at 111.76 76.2 0)
       (effects (font (size 1.27 1.27)) hide)
     )
@@
       (effects (font (size 1.27 1.27)) hide)
     )
-    (property "Manufacturer_Part_Number" "CL05B104KB54PNC" (id 4) (at 119.38 52.07 0)
+    (property "Manufacturer_Part_Number" "C1005X7R1H104KT000S" (id 4) (at 119.38 52.07 0)
       (effects (font (size 1.27 1.27)) hide)
     )
@@
       (effects (font (size 1.27 1.27)) hide)
     )
-    (property "Manufacturer_Part_Number" "CL05A225MQ5NSNC" (id 4) (at 107.95 52.07 0)
+    (property "Manufacturer_Part_Number" "ZRB157R61C225KE11D" (id 4) (at 107.95 52.07 0)
       (effects (font (size 1.27 1.27)) hide)
     )
