File: ICM42605.kicad_sch (KiCad schematic)
At the start: 3 parts, among them U7 ICM-42605

Commit message: Little fix
Parts:
- C13: Manufacturer_Part_Number (none) -> CL05B104KB54PNC
- C14: Manufacturer_Part_Number (none) -> CL05A225MQ5NSNC
Changed lines of the file:
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@@
+      (effects (font (size 1.27 1.27)) hide)
+    )
+    (property "Manufacturer_Part_Number" "CL05B104KB54PNC" (id 4) (at 125.73 68.58 0)
       (effects (font (size 1.27 1.27)) hide)
     )
@@
       (effects (font (size 1.27 1.27)) hide)
     )
+    (property "Manufacturer_Part_Number" "CL05A225MQ5NSNC" (id 4) (at 125.73 76.2 0)
+      (effects (font (size 1.27 1.27)) hide)
+    )

Commit message: First order
Parts:
- C13: Manufacturer_Part_Number CL05B104KB54PNC -> C1005X7R1H104KT000S
- C14: Manufacturer_Part_Number CL05A225MQ5NSNC -> ZRB157R61C225KE11D
Changed lines of the file:
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@@
       (effects (font (size 1.27 1.27)) hide)
     )
-    (property "Manufacturer_Part_Number" "CL05B104KB54PNC" (id 4) (at 125.73 68.58 0)
+    (property "Manufacturer_Part_Number" "C1005X7R1H104KT000S" (id 4) (at 125.73 68.58 0)
       (effects (font (size 1.27 1.27)) hide)
     )
@@
       (effects (font (size 1.27 1.27)) hide)
     )
-    (property "Manufacturer_Part_Number" "CL05A225MQ5NSNC" (id 4) (at 125.73 76.2 0)
+    (property "Manufacturer_Part_Number" "ZRB157R61C225KE11D" (id 4) (at 125.73 76.2 0)
       (effects (font (size 1.27 1.27)) hide)
     )
