File: Power.kicad_sch (KiCad schematic)
At the start: 9 parts, among them Q1 Si7336ADP, Q2 Si7336ADP, U12 U74AHC1G04G-AL5-R, U13 74LVC1G08GV, U14 NC7SZ02M5X

Commit message: плата практически готова
Parts:
- removed Q1, Q2: Si7336ADP, Package_SO:PowerPAK_SO-8_Single, symbol Transistor_FET:Si7336ADP
- removed R3: 100R, Resistor_SMD:R_0402_1005Metric, symbol Device:R
- removed U12: U74AHC1G04G-AL5-R, Package_TO_SOT_SMD:SOT-353_SC-70-5, symbol 74xGxx:74AHC1G04
- removed U13: 74LVC1G08GV, Package_TO_SOT_SMD:SOT-23-5, symbol 74xGxx:74LVC1G08
- removed U14: NC7SZ02M5X, Package_TO_SOT_SMD:SOT-23-5, symbol 74xGxx:74AHC1G02
- added C24, C25, C26, C27: 22uF, Capacitor_SMD:C_0402_1005Metric, symbol Device:C
- added C28, C39, C40, C41: 10uF, Capacitor_Tantalum_SMD:CP_EIA-3216-18_Kemet-A, symbol Device:C_Polarized
- added D7: 1N5819WS, Diode_SMD:D_SOD-323, symbol Device:D_Schottky
- added Q1: MMDT3906, Package_TO_SOT_SMD:SOT-363_SC-70-6, symbol Transistor_BJT:MMDT3906
- added Q2, Q8: DMP3013SFV, Package_SON:Diodes_PowerDI3333-8, symbol Transistor_FET:DMP3013SFV
- added Q4, Q5: AO3400A, Package_TO_SOT_SMD:SOT-23, symbol Transistor_FET:AO3400A
- added R47, R50: 220R, Resistor_SMD:R_0402_1005Metric, symbol Device:R
- added R54, R55, R56: 10K, Resistor_SMD:R_0402_1005Metric, symbol Device:R
- added U12, U9: AMS1117-3.3, Package_TO_SOT_SMD:SOT-223-3_TabPin2, symbol Regulator_Linear:AMS1117-3.3
- added U13: 74AHC1G04, Package_TO_SOT_SMD:SOT-353_SC-70-5, symbol 74xGxx:74AHC1G04
- R12: value 10K -> 1M
- R40: value 10K -> 100K
- R8: value 100R -> 220R
Connections:
- net GND: now also C24.1, C25.2, C26.2, C27.2, C28.2, C39.2, C40.2, C41.2, R54.1, R55.2, R56.2, U12.1 (GND), U13.3 (GND), U9.1 (GND)
- net VCC: now also C24.2, C39.1, C41.1, D7.1 (K), Q1.4 (E2), Q2.1 (S), Q2.2 (S), Q2.3 (S), Q4.3 (D), Q8.5 (D), U13.5 (VCC), U9.3 (VI)
- net at R12.1: now also Q1.2 (B1), Q1.5 (B2), Q1.6 (C1)
- net at R40.1: now also Q1.3 (C2), Q2.4 (G); no longer R8.1
- net PWR_EN3 renamed USB_SWITCH
- net USB_SWITCH: now also U13.2
- new net: Q4.1 (G), R50.2, R55.1
- new net: Q4.2 (S), Q5.2 (S)
- new net: Q5.1 (G), R54.2, R8.1
- new net: R50.1, U13.4
- new net 3V3_GROUP1: C26.1, C28.1, U9.2 (VO)
- new net 3V3_GROUP2: C27.1, C40.1, U12.2 (VO)
- new net 5V_GROUP2: C25.1, Q8.1 (S), Q8.2 (S), Q8.3 (S), U12.3 (VI)
- new net 5V_GROUP3: Q1.1 (E1), Q2.5 (D)
- new net GROUP2_EN: Q8.4 (G), R47.2, R56.1
- new net PWR_IN_JST: D7.2 (A)
- new net VBUS: Q5.3 (D), R47.1
Other:
- note added: "5V->3V3"
- note added: "DIODS"
- note added: "PWR EN"
- note removed: "FMU"
- note removed: "RPI CM4"

Commit message: Little fix
Parts:
- C24, C25, C26, C27: value 22uF -> 10uF; Manufacturer_Part_Number (none) -> CL31A226KAHNNNE
- Q8: Manufacturer_Part_Number (none) -> DMP3013SFV
- R12: Manufacturer_Part_Number (none) -> 0402WGF1004TCE
- R40: Manufacturer_Part_Number (none) -> 0402WGF100KTCE
- R47, R50, R8: Manufacturer_Part_Number (none) -> AECR0402F220RK9
- R54, R55, R56: Manufacturer_Part_Number (none) -> 0402WGF1002TCE
Changed lines of the file:
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@@
+      (effects (font (size 1.27 1.27)) hide)
+    )
+    (property "Manufacturer_Part_Number" "0402WGF1002TCE" (id 4) (at 133.35 109.22 0)
       (effects (font (size 1.27 1.27)) hide)
     )
@@
       (effects (font (size 1.27 1.27)) (justify left))
     )
-    (property "Value" "22uF" (id 1) (at 123.19 66.04 90)
+    (property "Value" "10uF" (id 1) (at 123.19 66.04 90)
       (effects (font (size 1.27 1.27)) (justify left))
     )
@@
     )
     (property "Datasheet" "~" (id 3) (at 127 62.23 0)
+      (effects (font (size 1.27 1.27)) hide)
+    )
+    (property "Manufacturer_Part_Number" "CL31A226KAHNNNE" (id 4) (at 127 62.23 0)
       (effects (font (size 1.27 1.27)) hide)
     )
@@
       (effects (font (size 1.27 1.27)) (justify left))
     )
-    (property "Value" "22uF" (id 1) (at 151.13 43.18 90)
+    (property "Value" "10uF" (id 1) (at 151.13 43.18 90)
       (effects (font (size 1.27 1.27)) (justify left))
     )
@@
       (effects (font (size 1.27 1.27)) hide)
     )
+    (property "Manufacturer_Part_Number" "CL31A226KAHNNNE" (id 4) (at 147.32 39.37 0)
+      (effects (font (size 1.27 1.27)) hide)
+    )
     (pin "1")
     (pin "2")
@@
       (effects (font (size 1.27 1.27)) (justify left))
     )
-    (property "Value" "22uF" (id 1) (at 151.13 66.04 90)
+    (property "Value" "10uF" (id 1) (at 151.13 66.04 90)
       (effects (font (size 1.27 1.27)) (justify left))
     )
@@
     )
     (property "Datasheet" "~" (id 3) (at 147.32 62.23 0)
+      (effects (font (size 1.27 1.27)) hide)
+    )
+    (property "Manufacturer_Part_Number" "CL31A226KAHNNNE" (id 4) (at 147.32 62.23 0)
       (effects (font (size 1.27 1.27)) hide)
     )
@@
       (effects (font (size 1.27 1.27)) hide)
     )
+    (property "Manufacturer_Part_Number" "AECR0402F220RK9" (id 4) (at 50.8 74.93 0)
+      (effects (font (size 1.27 1.27)) hide)
+    )
     (pin "1")
     (pin "2")
@@
       (effects (font (size 1.27 1.27)) hide)
     )
+    (property "Manufacturer_Part_Number" "0402WGF1002TCE" (id 4) (at 62.23 93.98 0)
+      (effects (font (size 1.27 1.27)) hide)
+    )
     (pin "1")
     (pin "2")
@@
       (effects (font (size 1.27 1.27)) hide)
     )
+    (property "Manufacturer_Part_Number" "0402WGF1002TCE" (id 4) (at 77.47 93.98 0)
+      (effects (font (size 1.27 1.27)) hide)
+    )
     (pin "1")
     (pin "2")
@@
       (effects (font (size 1.27 1.27)) hide)
     )
+    (property "Manufacturer_Part_Number" "AECR0402F220RK9" (id 4) (at 50.8 91.44 0)
+      (effects (font (size 1.27 1.27)) hide)
+    )
     (pin "1")
     (pin "2")
@@
       (effects (font (size 1.27 1.27)) hide)
     )
+    (property "Manufacturer_Part_Number" "0402WGF1004TCE" (id 4) (at 44.45 55.88 0)
+      (effects (font (size 1.27 1.27)) hide)
+    )
     (pin "1")
     (pin "2")
@@
     )
     (property "Datasheet" "~" (id 3) (at 50.8 86.36 0)
+      (effects (font (size 1.27 1.27)) hide)
+    )
+    (property "Manufacturer_Part_Number" "AECR0402F220RK9" (id 4) (at 50.8 86.36 0)
       (effects (font (size 1.27 1.27)) hide)
     )
@@
       (effects (font (size 1.27 1.27)) (justify left) hide)
     )
+    (property "Manufacturer_Part_Number" "DMP3013SFV" (id 4) (at 133.35 97.79 0)
+      (effects (font (size 1.27 1.27)) hide)
+    )
     (pin "1")
     (pin "2")
@@
       (effects (font (size 1.27 1.27)) (justify left))
     )
-    (property "Value" "22uF" (id 1) (at 123.19 38.1 90)
+    (property "Value" "10uF" (id 1) (at 123.19 38.1 90)
       (effects (font (size 1.27 1.27)) (justify left))
     )
@@
     )
     (property "Datasheet" "~" (id 3) (at 127 39.37 0)
+      (effects (font (size 1.27 1.27)) hide)
+    )
+    (property "Manufacturer_Part_Number" "CL31A226KAHNNNE" (id 4) (at 127 39.37 0)
       (effects (font (size 1.27 1.27)) hide)
     )
@@
       (effects (font (size 1.27 1.27)) hide)
     )
+    (property "Manufacturer_Part_Number" "0402WGF100KTCE" (id 4) (at 63.5 55.88 0)
+      (effects (font (size 1.27 1.27)) hide)
+    )

Commit message: First order
Parts:
- removed Q2, Q8: DMP3013SFV, Package_SON:Diodes_PowerDI3333-8, symbol Transistor_FET:DMP3013SFV
- added Q2, Q8: SSM6J507NU,LF, TRANS_SSM6J507NU,LF, symbol SSM6J507NU_LF:SSM6J507NU,LF
- C24, C25, C26, C27, C28, C39, C40, C41: Manufacturer_Part_Number CL31A226KAHNNNE -> CL05A106MP8NUB8
- D7: value 1N5819WS -> BAT60JFILM; Manufacturer_Part_Number 1N5819WS -> BAT60JFILM
- R12: Manufacturer_Part_Number 0402WGF1004TCE -> (none)
- R40: Manufacturer_Part_Number 0402WGF100KTCE -> PTFR0402B100KN9
- R47, R50, R8: Manufacturer_Part_Number AECR0402F220RK9 -> PTFR0402B220RP9
- R54, R55, R56: Manufacturer_Part_Number 0402WGF1002TCE -> RNCF0402BTE10K0
Connections:
- net 5V_GROUP2: now also Q8.4, Q8.8
- net 5V_GROUP3: now also Q2.1, Q2.2, Q2.5, Q2.6, Q2.7
- net GROUP2_EN: now also Q8.3
- net VCC: now also Q2.4, Q2.8, Q8.1, Q8.2, Q8.5, Q8.6, Q8.7
- net at Q1.3 (C2), R40.1: now also Q2.3
Other:
- moved on the sheet: R56
