File: RPi_CM4.kicad_sch (KiCad schematic)
At the start: 21 parts, among them J1 Micro_SD_Card, U16 CAT24C256, U6 Compute_Module_4_Connectors

Commit message: плата практически готова
Parts:
- removed J1: Micro_SD_Card, Connector_Card:microSD_HC_Wuerth_693072010801, symbol Connector:Micro_SD_Card
- added U21: 47579-0001, 47579-0001:POS-8, symbol 47579-0001:47579-0001
Connections:
- net RPI_I2C1_SCL is gone; now on net RPI_I2C1.SCL: U16.6 (SCL)
- net RPI_I2C1_SDA is gone; now on net RPI_I2C1.SDA: U16.5 (SDA)
- net GND: now also U21.G1 (GND), U21.G2 (GND), U21.P6 (VSS)
- net RPI_OUT_3V3: now also U21.P4 (VDD)
- net at R21.2: now also U21.P1 (DAT2)
- net at R1.2: now also U21.P2 (DAT3)
- net at R2.2: now also U21.P3 (CMD)
- net at R6.1: now also U21.P5 (CLK)
- net at R9.1: now also U21.P7 (DAT0)
- net at R10.1: now also U21.P8 (DAT1)
- net RPI_SD_PWR_ON: no longer names the net of U6.75 (SD_PWR_ON)
- no-connect marks 0 -> 103
Other:
- moved on the sheet: C17, C18, C35, JP2, R1, R10, R19, R2, R20, R21, R29, R34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

Commit message: )
Parts:
- JP2: footprint Jumper:SolderJumper-2_P1.3mm_Open_TrianglePad1.0x1.5mm -> Jumper:SolderJumper-2_P1.3mm_Open_RoundedPad1.0x1.5mm
Changed lines of the file:
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@@
     (property "Reference" "JP2" (id 0) (at 31.75 197.993 0))
     (property "Value" "BR" (id 1) (at 31.75 200.3044 0))
-    (property "Footprint" "Jumper:SolderJumper-2_P1.3mm_Open_TrianglePad1.0x1.5mm" (id 2) (at 31.75 203.2 0)
+    (property "Footprint" "Jumper:SolderJumper-2_P1.3mm_Open_RoundedPad1.0x1.5mm" (id 2) (at 31.75 203.2 0)
       (effects (font (size 1.27 1.27)) hide)
     )

Commit message: Little fix
Parts:
- C17, C18, C35: Manufacturer_Part_Number (none) -> CL05B104KB54PNC
- R1, R10, R2, R21, R6, R9: Manufacturer_Part_Number (none) -> 0402WGF330JTCE
- R19, R20, R29: Manufacturer_Part_Number (none) -> 0402WGF4701TCE
- R34: Manufacturer_Part_Number (none) -> 0402WGF5101TCE
- R35, R36, R37: Manufacturer_Part_Number (none) -> 0402WGF100KTCE
Connections:
- net GND: now also U16.9 (PAD)
- no-connect marks 103 -> 105
Changed lines of the file:
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@@
   (junction (at 236.22 129.54) (diameter 0) (color 0 0 0 0)
   )
-  (junction (at 53.34 140.97) (diameter 0) (color 0 0 0 0)
-  )
   (junction (at 238.76 114.3) (diameter 0) (color 0 0 0 0)
   )
@@
   )
   (junction (at 172.72 106.68) (diameter 0) (color 0 0 0 0)
+  )
+  (junction (at 53.34 143.51) (diameter 0) (color 0 0 0 0)
+  )
+  (junction (at 64.77 135.89) (diameter 0) (color 0 0 0 0)
   )
   (junction (at 172.72 83.82) (diameter 0) (color 0 0 0 0)
@@
   (no_connect (at 360.68 44.45))
   (no_connect (at 360.68 41.91))
+  (no_connect (at 43.18 73.66))
+  (no_connect (at 43.18 76.2))
   (no_connect (at 236.22 35.56))
   (no_connect (at 360.68 125.73))
@@
     (stroke (width 0) (type default) (color 0 0 0 0))
   )
+  (wire (pts (xy 63.5 135.89) (xy 64.77 135.89))
+    (stroke (width 0) (type default) (color 0 0 0 0))
+  )
   (wire (pts (xy 53.34 123.19) (xy 53.34 118.11))
     (stroke (width 0) (type default) (color 0 0 0 0))
@@
     (stroke (width 0) (type default) (color 0 0 0 0))
   )
-  (wire (pts (xy 64.77 133.35) (xy 64.77 140.97))
+  (wire (pts (xy 64.77 133.35) (xy 64.77 135.89))
     (stroke (width 0) (type default) (color 0 0 0 0))
   )
@@
     (stroke (width 0) (type default) (color 0 0 0 0))
   )
-  (wire (pts (xy 53.34 140.97) (xy 53.34 142.24))
-    (stroke (width 0) (type default) (color 0 0 0 0))
-  )
   (bus (pts (xy 43.18 185.42) (xy 43.18 187.96))
     (stroke (width 0) (type default) (color 0 0 0 0))
@@
     (stroke (width 0) (type default) (color 0 0 0 0))
   )
+  (wire (pts (xy 39.37 143.51) (xy 39.37 140.97))
+    (stroke (width 0) (type default) (color 0 0 0 0))
+  )
   (wire (pts (xy 360.68 107.95) (xy 363.22 107.95))
     (stroke (width 0) (type default) (color 0 0 0 0))
@@
     (stroke (width 0) (type default) (color 0 0 0 0))
   )
+  (wire (pts (xy 64.77 135.89) (xy 64.77 143.51))
+    (stroke (width 0) (type default) (color 0 0 0 0))
+  )
   (bus (pts (xy 383.54 69.85) (xy 383.54 64.77))
     (stroke (width 0) (type default) (color 0 0 0 0))
@@
     (stroke (width 0) (type default) (color 0 0 0 0))
   )
-  (wire (pts (xy 64.77 140.97) (xy 53.34 140.97))
+  (wire (pts (xy 64.77 143.51) (xy 53.34 143.51))
     (stroke (width 0) (type default) (color 0 0 0 0))
   )
@@
     (stroke (width 0) (type default) (color 0 0 0 0))
   )
-  (wire (pts (xy 53.34 138.43) (xy 53.34 140.97))
-    (stroke (width 0) (type default) (color 0 0 0 0))
-  )
   (wire (pts (xy 238.76 86.36) (xy 238.76 99.06))
     (stroke (width 0) (type default) (color 0 0 0 0))
@@
     (stroke (width 0) (type default) (color 0 0 0 0))
   )
+  (wire (pts (xy 53.34 143.51) (xy 53.34 144.78))
+    (stroke (width 0) (type default) (color 0 0 0 0))
+  )
   (wire (pts (xy 38.1 172.72) (xy 39.37 172.72))
     (stroke (width 0) (type default) (color 0 0 0 0))
@@
     (stroke (width 0) (type default) (color 0 0 0 0))
   )
-  (wire (pts (xy 39.37 140.97) (xy 53.34 140.97))
+  (wire (pts (xy 39.37 143.51) (xy 53.34 143.51))
     (stroke (width 0) (type default) (color 0 0 0 0))
   )
@@
   )
   (wire (pts (xy 236.22 134.62) (xy 236.22 137.16))
+    (stroke (width 0) (type default) (color 0 0 0 0))
+  )
+  (wire (pts (xy 53.34 143.51) (xy 53.34 140.97))
     (stroke (width 0) (type default) (color 0 0 0 0))
   )
@@
       (effects (font (size 1.27 1.27)) hide)
     )
+    (property "Manufacturer_Part_Number" "0402WGF330JTCE" (id 4) (at 38.1 66.04 0)
+      (effects (font (size 1.27 1.27)) hide)
+    )
     (pin "1")
     (pin "2")
@@
       (effects (font (size 1.27 1.27)) hide)
     )
+    (property "Manufacturer_Part_Number" "0402WGF4701TCE" (id 4) (at 39.37 176.53 0)
+      (effects (font (size 1.27 1.27)) hide)
+    )
     (pin "1")
     (pin "2")
@@
       (effects (font (size 1.27 1.27)) hide)
     )
+    (property "Manufacturer_Part_Number" "0402WGF4701TCE" (id 8) (at 36.83 176.53 0)
+      (effects (font (size 1.27 1.27)) hide)
+    )
     (pin "1")
     (pin "2")
@@
       (effects (font (size 1.27 1.27)) hide)
     )
+    (property "Manufacturer_Part_Number" "CL05B104KB54PNC" (id 4) (at 80.01 43.18 0)
+      (effects (font (size 1.27 1.27)) hide)
+    )
     (pin "1")
     (pin "2")
@@
     )
     (property "Datasheet" "~" (id 3) (at 74.93 43.18 0)
+      (effects (font (size 1.27 1.27)) hide)
+    )
+    (property "Manufacturer_Part_Number" "CL05B104KB54PNC" (id 4) (at 74.93 43.18 0)
       (effects (font (size 1.27 1.27)) hide)
     )
@@
     (pin "7")
     (pin "8")
+    (pin "9")
   )
   (symbol (lib_id "Device:R") (at 41.91 123.19 180) (unit 1)
@@
       (effects (font (size 1.27 1.27)) hide)
     )
+    (property "Manufacturer_Part_Number" "0402WGF100KTCE" (id 8) (at 41.91 123.19 0)
+      (effects (font (size 1.27 1.27)) hide)
+    )
     (pin "1")
     (pin "2")
@@
       (effects (font (size 1.27 1.27)) hide)
     )
+    (property "Manufacturer_Part_Number" "0402WGF100KTCE" (id 8) (at 35.56 137.16 0)
+      (effects (font (size 1.27 1.27)) hide)
+    )
     (pin "1")
     (pin "2")
@@
       (effects (font (size 1.27 1.27)) hide)
     )
+    (property "Manufacturer_Part_Number" "0402WGF100KTCE" (id 8) (at 39.37 137.16 0)
+      (effects (font (size 1.27 1.27)) hide)
+    )
     (pin "1")
     (pin "2")
   )
-  (symbol (lib_id "power:GND") (at 53.34 142.24 0) (unit 1)
-    (in_bom yes) (on_board yes)
-    (property "Reference" "#PWR06" (id 0) (at 53.34 148.59 0)
-      (effects (font (size 1.27 1.27)) hide)
-    )
-    (property "Value" "GND" (id 1) (at 53.467 146.6342 0))
-    (property "Footprint" "" (id 2) (at 53.34 142.24 0)
-      (effects (font (size 1.27 1.27)) hide)
-    )
-    (property "Datasheet" "" (id 3) (at 53.34 142.24 0)
+  (symbol (lib_id "power:GND") (at 53.34 144.78 0) (unit 1)
+    (in_bom yes) (on_board yes)
+    (property "Reference" "#PWR06" (id 0) (at 53.34 151.13 0)
+      (effects (font (size 1.27 1.27)) hide)
+    )
+    (property "Value" "GND" (id 1) (at 53.467 149.1742 0))
+    (property "Footprint" "" (id 2) (at 53.34 144.78 0)
+      (effects (font (size 1.27 1.27)) hide)
+    )
+    (property "Datasheet" "" (id 3) (at 53.34 144.78 0)
       (effects (font (size 1.27 1.27)) hide)
     )
@@
     )
     (property "Value" "100nF" (id 7) (at 33.02 123.19 0)
+      (effects (font (size 1.27 1.27)) hide)
+    )
+    (property "Manufacturer_Part_Number" "CL05B104KB54PNC" (id 8) (at 33.02 123.19 0)
       (effects (font (size 1.27 1.27)) hide)
     )
@@
     (in_bom yes) (on_board yes)
     (property "Reference" "R34" (id 0) (at 21.4122 208.28 90))
-    (property "Value" "1K5" (id 1) (at 23.7236 208.28 90))
+    (property "Value" "5K1" (id 1) (at 23.7236 208.28 90))
     (property "Footprint" "Resistor_SMD:R_0402_1005Metric" (id 2) (at 24.892 208.28 90)
       (effects (font (size 1.27 1.27)) hide)
@@
     )
     (property "Value" "1K5" (id 7) (at 26.67 208.28 0)
+      (effects (font (size 1.27 1.27)) hide)
+    )
+    (property "Manufacturer_Part_Number" "0402WGF5101TCE" (id 8) (at 26.67 208.28 0)
       (effects (font (size 1.27 1.27)) hide)
     )
@@
       (effects (font (size 1.27 1.27)) hide)
     )
+    (property "Manufacturer_Part_Number" "0402WGF330JTCE" (id 4) (at 31.75 68.58 0)
+      (effects (font (size 1.27 1.27)) hide)
+    )
     (pin "1")
     (pin "2")
@@
       (effects (font (size 1.27 1.27)) hide)
     )
+    (property "Manufacturer_Part_Number" "0402WGF330JTCE" (id 4) (at 38.1 43.18 0)
+      (effects (font (size 1.27 1.27)) hide)
+    )
     (pin "1")
     (pin "2")
@@
     )
     (property "Datasheet" "~" (id 3) (at 38.1 45.72 0)
+      (effects (font (size 1.27 1.27)) hide)
+    )
+    (property "Manufacturer_Part_Number" "0402WGF330JTCE" (id 4) (at 38.1 45.72 0)
       (effects (font (size 1.27 1.27)) hide)
     )
@@
       (effects (font (size 1.27 1.27)) hide)
     )
+    (property "Manufacturer_Part_Number" "0402WGF4701TCE" (id 8) (at 74.93 176.53 0)
+      (effects (font (size 1.27 1.27)) hide)
+    )
     (pin "1")
     (pin "2")
@@
       (effects (font (size 1.27 1.27)) hide)
     )
+    (property "Manufacturer_Part_Number" "0402WGF330JTCE" (id 4) (at 38.1 63.5 0)
+      (effects (font (size 1.27 1.27)) hide)
+    )
     (pin "1")
     (pin "2")
@@
       (effects (font (size 1.27 1.27)) hide)
     )
+    (property "Manufacturer_Part_Number" "0402WGF330JTCE" (id 4) (at 31.75 60.96 0)
+      (effects (font (size 1.27 1.27)) hide)
+    )
     (pin "1")
     (pin "2")
@@
       (effects (font (size 1.27 1.27)) hide)
     )
+    (property "Manufacturer_Part_Number" "0402WGF4701TCE" (id 4) (at 77.47 176.53 0)
+      (effects (font (size 1.27 1.27)) hide)
+    )

Commit message: First order
Parts:
- C17, C18, C35: Manufacturer_Part_Number CL05B104KB54PNC -> C1005X7R1H104KT000S
- R1, R10, R2, R21, R6, R9: Manufacturer_Part_Number 0402WGF330JTCE -> (none)
- R19, R20, R29: Manufacturer_Part_Number 0402WGF4701TCE -> ERJPA2F4701X
- R34: Manufacturer_Part_Number 0402WGF5101TCE -> PTFR0402B5K10N9
- R35, R36, R37: Manufacturer_Part_Number 0402WGF100KTCE -> PTFR0402B100KN9
Changed lines of the file:
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@@
       (effects (font (size 1.27 1.27)) hide)
     )
-    (property "Manufacturer_Part_Number" "0402WGF330JTCE" (id 4) (at 38.1 66.04 0)
+    (property "Manufacturer_Part_Number" "" (id 4) (at 38.1 66.04 0)
       (effects (font (size 1.27 1.27)) hide)
     )
@@
       (effects (font (size 1.27 1.27)) hide)
     )
-    (property "Manufacturer_Part_Number" "0402WGF4701TCE" (id 4) (at 39.37 176.53 0)
+    (property "Manufacturer_Part_Number" "ERJPA2F4701X" (id 4) (at 39.37 176.53 0)
       (effects (font (size 1.27 1.27)) hide)
     )
@@
       (effects (font (size 1.27 1.27)) hide)
     )
-    (property "Manufacturer_Part_Number" "0402WGF4701TCE" (id 8) (at 36.83 176.53 0)
+    (property "Manufacturer_Part_Number" "ERJPA2F4701X" (id 8) (at 36.83 176.53 0)
       (effects (font (size 1.27 1.27)) hide)
     )
@@
       (effects (font (size 1.27 1.27)) hide)
     )
-    (property "Manufacturer_Part_Number" "CL05B104KB54PNC" (id 4) (at 80.01 43.18 0)
+    (property "Manufacturer_Part_Number" "C1005X7R1H104KT000S" (id 4) (at 80.01 43.18 0)
       (effects (font (size 1.27 1.27)) hide)
     )
@@
       (effects (font (size 1.27 1.27)) hide)
     )
-    (property "Manufacturer_Part_Number" "CL05B104KB54PNC" (id 4) (at 74.93 43.18 0)
+    (property "Manufacturer_Part_Number" "C1005X7R1H104KT000S" (id 4) (at 74.93 43.18 0)
       (effects (font (size 1.27 1.27)) hide)
     )
@@
       (effects (font (size 1.27 1.27)) hide)
     )
-    (property "Manufacturer_Part_Number" "0402WGF100KTCE" (id 8) (at 41.91 123.19 0)
+    (property "Manufacturer_Part_Number" "PTFR0402B100KN9" (id 8) (at 41.91 123.19 0)
       (effects (font (size 1.27 1.27)) hide)
     )
@@
       (effects (font (size 1.27 1.27)) hide)
     )
-    (property "Manufacturer_Part_Number" "0402WGF100KTCE" (id 8) (at 35.56 137.16 0)
+    (property "Manufacturer_Part_Number" "PTFR0402B100KN9" (id 8) (at 35.56 137.16 0)
       (effects (font (size 1.27 1.27)) hide)
     )
@@
       (effects (font (size 1.27 1.27)) hide)
     )
-    (property "Manufacturer_Part_Number" "0402WGF100KTCE" (id 8) (at 39.37 137.16 0)
+    (property "Manufacturer_Part_Number" "PTFR0402B100KN9" (id 8) (at 39.37 137.16 0)
       (effects (font (size 1.27 1.27)) hide)
     )
@@
       (effects (font (size 1.27 1.27)) hide)
     )
-    (property "Manufacturer_Part_Number" "CL05B104KB54PNC" (id 8) (at 33.02 123.19 0)
+    (property "Manufacturer_Part_Number" "C1005X7R1H104KT000S" (id 8) (at 33.02 123.19 0)
       (effects (font (size 1.27 1.27)) hide)
     )
@@
       (effects (font (size 1.27 1.27)) hide)
     )
-    (property "Manufacturer_Part_Number" "0402WGF5101TCE" (id 8) (at 26.67 208.28 0)
+    (property "Manufacturer_Part_Number" "PTFR0402B5K10N9" (id 8) (at 26.67 208.28 0)
       (effects (font (size 1.27 1.27)) hide)
     )
@@
       (effects (font (size 1.27 1.27)) hide)
     )
-    (property "Manufacturer_Part_Number" "0402WGF330JTCE" (id 4) (at 31.75 68.58 0)
+    (property "Manufacturer_Part_Number" "" (id 4) (at 31.75 68.58 0)
       (effects (font (size 1.27 1.27)) hide)
     )
@@
       (effects (font (size 1.27 1.27)) hide)
     )
-    (property "Manufacturer_Part_Number" "0402WGF330JTCE" (id 4) (at 38.1 43.18 0)
+    (property "Manufacturer_Part_Number" "" (id 4) (at 38.1 43.18 0)
       (effects (font (size 1.27 1.27)) hide)
     )
@@
       (effects (font (size 1.27 1.27)) hide)
     )
-    (property "Manufacturer_Part_Number" "0402WGF330JTCE" (id 4) (at 38.1 45.72 0)
+    (property "Manufacturer_Part_Number" "" (id 4) (at 38.1 45.72 0)
       (effects (font (size 1.27 1.27)) hide)
     )
@@
       (effects (font (size 1.27 1.27)) hide)
     )
-    (property "Manufacturer_Part_Number" "0402WGF4701TCE" (id 8) (at 74.93 176.53 0)
+    (property "Manufacturer_Part_Number" "ERJPA2F4701X" (id 8) (at 74.93 176.53 0)
       (effects (font (size 1.27 1.27)) hide)
     )
@@
       (effects (font (size 1.27 1.27)) hide)
     )
-    (property "Manufacturer_Part_Number" "0402WGF330JTCE" (id 4) (at 38.1 63.5 0)
+    (property "Manufacturer_Part_Number" "" (id 4) (at 38.1 63.5 0)
       (effects (font (size 1.27 1.27)) hide)
     )
@@
       (effects (font (size 1.27 1.27)) hide)
     )
-    (property "Manufacturer_Part_Number" "0402WGF330JTCE" (id 4) (at 31.75 60.96 0)
+    (property "Manufacturer_Part_Number" "" (id 4) (at 31.75 60.96 0)
       (effects (font (size 1.27 1.27)) hide)
     )
@@
       (effects (font (size 1.27 1.27)) hide)
     )
-    (property "Manufacturer_Part_Number" "0402WGF4701TCE" (id 4) (at 77.47 176.53 0)
-      (effects (font (size 1.27 1.27)) hide)
-    )
+    (property "Manufacturer_Part_Number" "ERJPA2F4701X" (id 4) (at 77.47 176.53 0)
+      (effects (font (size 1.27 1.27)) hide)
+    )
