File: STM32.kicad_sch (KiCad schematic)
At the start: 36 parts, among them U1 STM32H753IIKx, U4 FM25V02A-GTR, Y2 32.768

Commit message: плата практически готова
Parts:
- removed D1: LED_B, symbol Device:LED
- removed D2: LED_G, symbol Device:LED
- removed D3: LED_R, symbol Device:LED
- removed F1: Fuse, Fuse:Fuse_0603_1608Metric, symbol Device:Fuse
- removed U?: MIC2026-2BM, symbol Power_Management:MIC2026-2BM
- removed Y?: 16MHz, Crystal:Crystal_SMD_2016-4Pin_2.0x1.6mm, symbol Device:Crystal_GND23
- added D1: LED_RBAG, LED_SMD:LED_Cree-PLCC4_2x2mm_CW, symbol Device:LED_RBAG
- added D5: 1N5819WS, Diode_SMD:D_SOD-323, symbol Device:D_Schottky
- added Q6: 2N7002K, Package_TO_SOT_SMD:SOT-23, symbol Transistor_FET:2N7002K
- added Q7: FDN340P, Package_TO_SOT_SMD:SOT-23, symbol Transistor_FET:FDN340P
- added Y1: 16MHz, Crystal:Crystal_SMD_2016-4Pin_2.0x1.6mm, symbol Device:Crystal_GND24
- gave numbers to parts that had none: 4
Connections:
- net GND: now also R43.2, U1.D5 (VSS), U1.D7 (VSS), U1.D8 (VSS), U1.D9 (VSS), U1.F10 (VSS), U1.F12 (VSS), U1.F2 (VSS), U1.F6 (VSS), U1.F7 (VSS), U1.F8 (VSS), U1.F9 (VSS), U1.G12 (VSS), U1.G2 (VSS), U1.G6 (VSS), U1.G7 (VSS), U1.G8 (VSS), U1.G9 (VSS), U1.H10 (VSS), U1.H12 (VSS), U1.H6 (VSS), U1.H7 (VSS), U1.H8 (VSS), U1.H9 (VSS), U1.J10 (VSS), U1.J6 (VSS), U1.J7 (VSS), U1.J8 (VSS), U1.J9 (VSS), U1.K10 (VSS), U1.K6 (VSS), U1.K7 (VSS), U1.K8 (VSS), U1.K9 (VSS), U1.L4 (VSS), U1.M1 (VSSA), U1.M8 (VSS), U1.M9 (VSS), Q6.2 (S), Y1.2, Y1.4
- net SENSORS_3V3: now also Q7.3 (D)
- net STM_16MHZ_IN: now also Y1.1
- net STM_16MHZ_OUT: now also Y1.3
- net STM_3V3: now also R44.1, D1.3 (A), D5.1 (K), Q7.2 (S); no longer R43.1, R44.2
- net STM_NLED_GREEN: now also R32.2; no longer R32.1
- net STM_VDD_3V3_SENSORS_EN: now also R43.1, Q6.1 (G)
- net at R31.2: now also D1.1 (RK)
- net at R33.2: now also D1.2 (BK)
- new net: D1.4 (GK), R32.1
- new net: Q6.3 (D), Q7.1 (G), R44.2
- new net STM_DEBUG.3V3: D5.2 (A)
Other:
- moved on the sheet: C1, C10, C2, JP1, R11, R13, R22, R23, R24, R25, R26, R27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

Commit message: )
Parts:
- JP1: footprint Jumper:SolderJumper-2_P1.3mm_Open_TrianglePad1.0x1.5mm -> Jumper:SolderJumper-2_P1.3mm_Open_RoundedPad1.0x1.5mm
Connections:
- net STM_5V_HIPOWER_NOC: no longer names the net of U1.N6 (PF13)
- net STM_5V_PERIPH_NOC: no longer names the net of U1.R11 (PE15)
- net STM_BUZZER_1: no longer names the net of U1.L2 (PF9)
- net STM_CAN1_RX: no longer names the net of U1.B12 (PD0)
- net STM_CAN1_TX: no longer names the net of U1.C12 (PD1)
- net STM_CAP1: no longer names the net of U1.P10 (PE11)
- net STM_CAP2: no longer names the net of U1.N2 (PA1)
- net STM_HEATER: no longer names the net of U1.P2 (PA2)
- net STM_MUX_CTRL1: no longer names the net of U1.P5 (PC5)
- net STM_MUX_CTRL2: no longer names the net of U1.R8 (PE7)
- net STM_NARMED: no longer names the net of U1.B3 (PE6)
- net STM_NFC_GPIO: no longer names the net of U1.P6 (PF12)
- net STM_NPOWER_IN_A: no longer names the net of U1.M7 (PG1)
- net STM_NPOWER_IN_B: no longer names the net of U1.L15 (PG2)
- net STM_NPOWER_IN_C: no longer names the net of U1.K15 (PG3)
- net STM_NSAFETY_SWITCH_LED_OUT: no longer names the net of U1.N15 (PD10)
- net STM_PD15: no longer names the net of U1.L14 (PD15)
- net STM_PF4: no longer names the net of U1.J3 (PF4)
- net STM_PG15: no longer names the net of U1.B7 (PG15)
- net STM_PG6: no longer names the net of U1.J15 (PG6)
- net STM_PG8: no longer names the net of U1.H14 (PG8)
- net STM_SAFETY_SWITCH_IN: no longer names the net of U1.K3 (PF5)
- net STM_SDMMC2_CLK: no longer names the net of U1.M3 (PC1)
- net STM_SDMMC2_CMD: no longer names the net of U1.A11 (PD7)
- net STM_SDMMC2_D0: no longer names the net of U1.R14 (PB14)
- net STM_SDMMC2_D1: no longer names the net of U1.R15 (PB15)
- net STM_SDMMC2_D2: no longer names the net of U1.A10 (PB3)
- net STM_SDMMC2_D3: no longer names the net of U1.A9 (PB4)
- net STM_SPIX_SYNC: no longer names the net of U1.P9 (PE9)
- net STM_TRACECLK: no longer names the net of U1.A2 (PE2)
- net STM_V5_SCALED: no longer names the net of U1.N3 (PA0)
- net STM_VDD_3V3_SD_EN: no longer names the net of U1.D1 (PC13)
- net STM_VDD_5V_HIPOWER_NEN: no longer names the net of U1.B10 (PG10)
- net STM_VDD_5V_PERIPH_NEN: no longer names the net of U1.K14 (PG4)
- no-connect marks 0 -> 34

Commit message: тестирование
Connections:
- net STM_I2C2.SCL: no longer names the net of U1.H3 (PF1)
- net STM_I2C2.SDA: no longer names the net of U1.E2 (PF0)
- net STM_I2C3.SCL: no longer names the net of U1.F15 (PA8)
- net STM_I2C3.SDA: no longer names the net of U1.M12 (PH8)
- net STM_OTG_HS_ULPI_CK: no longer names the net of U1.P4 (PA5)
- net STM_OTG_HS_ULPI_D0: no longer names the net of U1.R2 (PA3)
- net STM_OTG_HS_ULPI_D1: no longer names the net of U1.R5 (PB0)
- net STM_OTG_HS_ULPI_D2: no longer names the net of U1.R4 (PB1)
- net STM_OTG_HS_ULPI_D3: no longer names the net of U1.R12 (PB10)
- net STM_OTG_HS_ULPI_D4: no longer names the net of U1.R13 (PB11)
- net STM_OTG_HS_ULPI_D5: no longer names the net of U1.P12 (PB12)
- net STM_OTG_HS_ULPI_D6: no longer names the net of U1.P13 (PB13)
- net STM_OTG_HS_ULPI_D7: no longer names the net of U1.A6 (PB5)
- net STM_OTG_HS_ULPI_DIR: no longer names the net of U1.E4 (PI11)
- net STM_OTG_HS_ULPI_NXT: no longer names the net of U1.M5 (PC3_C)
- net STM_OTG_HS_ULPI_STP: no longer names the net of U1.M2 (PC0)
- net STM_SPI4.CS1: no longer names the net of U1.D13 (PH15)
- net STM_SPI4.MISO: no longer names the net of U1.N11 (PE13)
- net STM_SPI4.MOSI: no longer names the net of U1.P11 (PE14)
- net STM_SPI4.SCK: no longer names the net of U1.R10 (PE12)
- net STM_SPI6.CS1: no longer names the net of U1.E3 (PI10)
- net STM_SPI6.CS2: no longer names the net of U1.A13 (PA15)
- net STM_SPI6.DRDY1: no longer names the net of U1.N14 (PD11)
- net STM_SPI6.DRDY2: no longer names the net of U1.N13 (PD12)
- net STM_SPI6.MISO: no longer names the net of U1.P3 (PA6)
- net STM_SPI6.MOSI: no longer names the net of U1.A7 (PG14)
- net STM_SPI6.NRESET: no longer names the net of U1.L1 (PF10)
- net STM_SPI6.SCK: no longer names the net of U1.A8 (PG13)
- net STM_UART4.RX: no longer names the net of U1.E13 (PH14)
- net STM_UART4.TX: no longer names the net of U1.E12 (PH13)
- net STM_UART8.RX: no longer names the net of U1.A4 (PE0)
- net STM_UART8.TX: no longer names the net of U1.A3 (PE1)
- no-connect marks 34 -> 66

Commit message: second version
Connections:
- net STM_UART5.CTS: no longer names the net of U1.F14 (PC9)
- net STM_UART5.RTS: no longer names the net of U1.G14 (PC8)
- net STM_UART7.CTS: no longer names the net of U1.R9 (PE10)
- net STM_UART7.RTS: no longer names the net of U1.L3 (PF8)
- net STM_USART2.CTS: no longer names the net of U1.D11 (PD3)
- net STM_USART2.RTS: no longer names the net of U1.D10 (PD4)
- no-connect marks 66 -> 72

Commit message: первый релиз
Parts:
- added R57: 220R, Resistor_SMD:R_0402_1005Metric, symbol Device:R
Connections:
- net STM_VDD_3V3_SENSORS_EN: now also R57.2; no longer Q6.1 (G), R43.1
- new net: Q6.1 (G), R43.1, R57.1
Other:
- moved on the sheet: Q6, Q7, R43, R44

Commit message: Little fix
Parts:
- C1, C2: Manufacturer_Part_Number (none) -> CL05A225MQ5NSNC
- C10: Manufacturer_Part_Number (none) -> CL05B104KB54PNC
- C11, C8: Manufacturer_Part_Number (none) -> 0402CG150J500NT
- C12, C9: Manufacturer_Part_Number (none) -> 0402CG120J500NT
- R13, R22: Manufacturer_Part_Number (none) -> 0402WGF4701TCE
- R23, R24, R28, R4, R43, R44, R45, R46, R5: Manufacturer_Part_Number (none) -> 0402WGF1002TCE
- R31, R32, R33: Manufacturer_Part_Number (none) -> 0402WGF1000TCE
- R57: Manufacturer_Part_Number (none) -> AECR0402F220RK9
- R7: Manufacturer_Part_Number (none) -> 0402WGF100KTCE
Changed lines of the file:
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@@
+      (effects (font (size 1.27 1.27)) hide)
+    )
+    (property "Manufacturer_Part_Number" "0402WGF1002TCE" (id 4) (at 41.91 39.37 0)
       (effects (font (size 1.27 1.27)) hide)
     )
@@
       (effects (font (size 1.27 1.27)) hide)
     )
+    (property "Manufacturer_Part_Number" "0402WGF1002TCE" (id 4) (at 34.29 39.37 0)
+      (effects (font (size 1.27 1.27)) hide)
+    )
     (pin "1")
     (pin "2")
@@
       (effects (font (size 1.27 1.27)) hide)
     )
+    (property "Manufacturer_Part_Number" "0402WGF100KTCE" (id 4) (at 35.56 332.74 0)
+      (effects (font (size 1.27 1.27)) hide)
+    )
     (pin "1")
     (pin "2")
@@
     )
     (property "Datasheet" "~" (id 3) (at 35.56 346.71 0)
+      (effects (font (size 1.27 1.27)) hide)
+    )
+    (property "Manufacturer_Part_Number" "CL05B104KB54PNC" (id 4) (at 35.56 346.71 0)
       (effects (font (size 1.27 1.27)) hide)
     )
@@
       (effects (font (size 1.27 1.27)) hide)
     )
+    (property "Manufacturer_Part_Number" "0402CG150J500NT" (id 4) (at 57.15 154.94 0)
+      (effects (font (size 1.27 1.27)) hide)
+    )
     (pin "1")
     (pin "2")
@@
     )
     (property "Datasheet" "~" (id 3) (at 39.37 154.94 0)
+      (effects (font (size 1.27 1.27)) hide)
+    )
+    (property "Manufacturer_Part_Number" "0402CG150J500NT" (id 4) (at 39.37 154.94 0)
       (effects (font (size 1.27 1.27)) hide)
     )
@@
       (effects (font (size 1.27 1.27)) hide)
     )
+    (property "Manufacturer_Part_Number" "0402CG120J500NT" (id 4) (at 54.61 177.8 0)
+      (effects (font (size 1.27 1.27)) hide)
+    )
     (pin "1")
     (pin "2")
@@
     )
     (property "Datasheet" "~" (id 3) (at 41.91 177.8 0)
+      (effects (font (size 1.27 1.27)) hide)
+    )
+    (property "Manufacturer_Part_Number" "0402CG120J500NT" (id 4) (at 41.91 177.8 0)
       (effects (font (size 1.27 1.27)) hide)
     )
@@
       (effects (font (size 1.27 1.27)) hide)
     )
+    (property "Manufacturer_Part_Number" "0402WGF1000TCE" (id 4) (at 53.34 96.52 0)
+      (effects (font (size 1.27 1.27)) hide)
+    )
     (pin "1")
     (pin "2")
@@
       (effects (font (size 1.27 1.27)) hide)
     )
+    (property "Manufacturer_Part_Number" "0402WGF1000TCE" (id 4) (at 53.34 104.14 0)
+      (effects (font (size 1.27 1.27)) hide)
+    )
     (pin "1")
     (pin "2")
@@
       (effects (font (size 1.27 1.27)) hide)
     )
+    (property "Manufacturer_Part_Number" "0402WGF1000TCE" (id 4) (at 53.34 111.76 0)
+      (effects (font (size 1.27 1.27)) hide)
+    )
     (pin "1")
     (pin "2")
@@
       (effects (font (size 1.27 1.27)) hide)
     )
+    (property "Manufacturer_Part_Number" "0402WGF1002TCE" (id 4) (at 62.23 212.09 0)
+      (effects (font (size 1.27 1.27)) hide)
+    )
     (pin "1")
     (pin "2")
@@
       (effects (font (size 1.27 1.27)) hide)
     )
+    (property "Manufacturer_Part_Number" "0402WGF1002TCE" (id 4) (at 58.42 273.05 0)
+      (effects (font (size 1.27 1.27)) hide)
+    )
     (pin "1")
     (pin "2")
@@
       (effects (font (size 1.27 1.27)) hide)
     )
+    (property "Manufacturer_Part_Number" "0402WGF1002TCE" (id 4) (at 45.72 339.09 0)
+      (effects (font (size 1.27 1.27)) hide)
+    )
     (pin "1")
     (pin "2")
@@
       (effects (font (size 1.27 1.27)) hide)
     )
+    (property "Manufacturer_Part_Number" "0402WGF4701TCE" (id 4) (at 49.53 267.335 0)
+      (effects (font (size 1.27 1.27)) hide)
+    )
     (pin "1")
     (pin "2")
@@
       (effects (font (size 1.27 1.27)) hide)
     )
+    (property "Manufacturer_Part_Number" "0402WGF1002TCE" (id 4) (at 35.56 325.12 0)
+      (effects (font (size 1.27 1.27)) hide)
+    )
     (pin "1")
     (pin "2")
@@
     )
     (property "Datasheet" "~" (id 3) (at 16.51 269.875 0)
+      (effects (font (size 1.27 1.27)) hide)
+    )
+    (property "Manufacturer_Part_Number" "CL05A225MQ5NSNC" (id 4) (at 16.51 269.875 0)
       (effects (font (size 1.27 1.27)) hide)
     )
@@
       (effects (font (size 1.27 1.27)) hide)
     )
+    (property "Manufacturer_Part_Number" "0402WGF4701TCE" (id 4) (at 41.91 267.335 0)
+      (effects (font (size 1.27 1.27)) hide)
+    )
     (pin "1")
     (pin "2")
@@
     )
     (property "Datasheet" "~" (id 3) (at 46.99 226.06 0)
+      (effects (font (size 1.27 1.27)) hide)
+    )
+    (property "Manufacturer_Part_Number" "AECR0402F220RK9" (id 4) (at 46.99 226.06 0)
       (effects (font (size 1.27 1.27)) hide)
     )
@@
       (effects (font (size 1.27 1.27)) hide)
     )
+    (property "Manufacturer_Part_Number" "0402WGF1002TCE" (id 4) (at 53.34 231.14 0)
+      (effects (font (size 1.27 1.27)) hide)
+    )
     (pin "1")
     (pin "2")
@@
       (effects (font (size 1.27 1.27)) hide)
     )
+    (property "Manufacturer_Part_Number" "0402WGF1002TCE" (id 4) (at 35.56 317.5 0)
+      (effects (font (size 1.27 1.27)) hide)
+    )
     (pin "1")
     (pin "2")
@@
     )
     (property "Datasheet" "~" (id 3) (at 58.42 257.81 0)
+      (effects (font (size 1.27 1.27)) hide)
+    )
+    (property "Manufacturer_Part_Number" "0402WGF1002TCE" (id 4) (at 58.42 257.81 0)
       (effects (font (size 1.27 1.27)) hide)
     )
@@
       (effects (font (size 1.27 1.27)) hide)
     )
+    (property "Manufacturer_Part_Number" "CL05A225MQ5NSNC" (id 4) (at 26.67 269.875 0)
+      (effects (font (size 1.27 1.27)) hide)
+    )

Commit message: First order
Parts:
- C1, C2: Manufacturer_Part_Number CL05A225MQ5NSNC -> ZRB157R61C225KE11D
- C10: Manufacturer_Part_Number CL05B104KB54PNC -> C1005X7R1H104KT000S
- C11, C8: Manufacturer_Part_Number 0402CG150J500NT -> GJM1555C1H150GB01D
- C12, C9: Manufacturer_Part_Number 0402CG120J500NT -> GCQ1555C1H120FB01D
- D5: value 1N5819WS -> BAT60JFILM; Manufacturer_Part_Number 1N5819WS -> BAT60JFILM
- R13, R22: Manufacturer_Part_Number 0402WGF4701TCE -> ERJPA2F4701X
- R23, R24, R28, R4, R43, R44, R45, R46, R5: Manufacturer_Part_Number 0402WGF1002TCE -> RNCF0402BTE10K0
- R31, R32, R33: Manufacturer_Part_Number 0402WGF1000TCE -> PTFR0402B100RN9
- R57: Manufacturer_Part_Number AECR0402F220RK9 -> PTFR0402B220RP9
- R7: Manufacturer_Part_Number 0402WGF100KTCE -> PTFR0402B100KN9
- Y2: Manufacturer_Part_Number SC-16S -> TFX-04-32.768K
Changed lines of the file:
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@@
       (effects (font (size 1.27 1.27)) hide)
     )
-    (property "Manufacturer_Part_Number" "0402WGF1002TCE" (id 4) (at 41.91 39.37 0)
+    (property "Manufacturer_Part_Number" "RNCF0402BTE10K0" (id 4) (at 41.91 39.37 0)
       (effects (font (size 1.27 1.27)) hide)
     )
@@
       (effects (font (size 1.27 1.27)) hide)
     )
-    (property "Manufacturer_Part_Number" "0402WGF1002TCE" (id 4) (at 34.29 39.37 0)
+    (property "Manufacturer_Part_Number" "RNCF0402BTE10K0" (id 4) (at 34.29 39.37 0)
       (effects (font (size 1.27 1.27)) hide)
     )
@@
       (effects (font (size 1.27 1.27)) hide)
     )
-    (property "Manufacturer_Part_Number" "0402WGF100KTCE" (id 4) (at 35.56 332.74 0)
+    (property "Manufacturer_Part_Number" "PTFR0402B100KN9" (id 4) (at 35.56 332.74 0)
       (effects (font (size 1.27 1.27)) hide)
     )
@@
       (effects (font (size 1.27 1.27)) hide)
     )
-    (property "Manufacturer_Part_Number" "CL05B104KB54PNC" (id 4) (at 35.56 346.71 0)
+    (property "Manufacturer_Part_Number" "C1005X7R1H104KT000S" (id 4) (at 35.56 346.71 0)
       (effects (font (size 1.27 1.27)) hide)
     )
@@
       (effects (font (size 1.27 1.27)) hide)
     )
-    (property "Manufacturer_Part_Number" "0402CG150J500NT" (id 4) (at 57.15 154.94 0)
+    (property "Manufacturer_Part_Number" "GJM1555C1H150GB01D" (id 4) (at 57.15 154.94 0)
       (effects (font (size 1.27 1.27)) hide)
     )
@@
       (effects (font (size 1.27 1.27)) hide)
     )
-    (property "Manufacturer_Part_Number" "0402CG150J500NT" (id 4) (at 39.37 154.94 0)
+    (property "Manufacturer_Part_Number" "GJM1555C1H150GB01D" (id 4) (at 39.37 154.94 0)
       (effects (font (size 1.27 1.27)) hide)
     )
@@
       (effects (font (size 1.27 1.27)) hide)
     )
-    (property "Manufacturer_Part_Number" "SC-16S" (id 4) (at 48.26 173.99 0)
+    (property "Manufacturer_Part_Number" "TFX-04-32.768K" (id 4) (at 48.26 173.99 0)
       (effects (font (size 1.27 1.27)) hide)
     )
@@
       (effects (font (size 1.27 1.27)) hide)
     )
-    (property "Manufacturer_Part_Number" "0402CG120J500NT" (id 4) (at 54.61 177.8 0)
+    (property "Manufacturer_Part_Number" "GCQ1555C1H120FB01D" (id 4) (at 54.61 177.8 0)
       (effects (font (size 1.27 1.27)) hide)
     )
@@
       (effects (font (size 1.27 1.27)) hide)
     )
-    (property "Manufacturer_Part_Number" "0402CG120J500NT" (id 4) (at 41.91 177.8 0)
+    (property "Manufacturer_Part_Number" "GCQ1555C1H120FB01D" (id 4) (at 41.91 177.8 0)
       (effects (font (size 1.27 1.27)) hide)
     )
@@
       (effects (font (size 1.27 1.27)) hide)
     )
-    (property "Manufacturer_Part_Number" "0402WGF1000TCE" (id 4) (at 53.34 96.52 0)
+    (property "Manufacturer_Part_Number" "PTFR0402B100RN9" (id 4) (at 53.34 96.52 0)
       (effects (font (size 1.27 1.27)) hide)
     )
@@
       (effects (font (size 1.27 1.27)) hide)
     )
-    (property "Manufacturer_Part_Number" "0402WGF1000TCE" (id 4) (at 53.34 104.14 0)
+    (property "Manufacturer_Part_Number" "PTFR0402B100RN9" (id 4) (at 53.34 104.14 0)
       (effects (font (size 1.27 1.27)) hide)
     )
@@
       (effects (font (size 1.27 1.27)) hide)
     )
-    (property "Manufacturer_Part_Number" "0402WGF1000TCE" (id 4) (at 53.34 111.76 0)
+    (property "Manufacturer_Part_Number" "PTFR0402B100RN9" (id 4) (at 53.34 111.76 0)
       (effects (font (size 1.27 1.27)) hide)
     )
@@
       (effects (font (size 1.27 1.27)) hide)
     )
-    (property "Manufacturer_Part_Number" "0402WGF1002TCE" (id 4) (at 62.23 212.09 0)
+    (property "Manufacturer_Part_Number" "RNCF0402BTE10K0" (id 4) (at 62.23 212.09 0)
       (effects (font (size 1.27 1.27)) hide)
     )
@@
       (effects (font (size 1.27 1.27)) hide)
     )
-    (property "Manufacturer_Part_Number" "0402WGF1002TCE" (id 4) (at 58.42 273.05 0)
+    (property "Manufacturer_Part_Number" "RNCF0402BTE10K0" (id 4) (at 58.42 273.05 0)
       (effects (font (size 1.27 1.27)) hide)
     )
@@
       (effects (font (size 1.27 1.27)) hide)
     )
-    (property "Manufacturer_Part_Number" "0402WGF1002TCE" (id 4) (at 45.72 339.09 0)
+    (property "Manufacturer_Part_Number" "RNCF0402BTE10K0" (id 4) (at 45.72 339.09 0)
       (effects (font (size 1.27 1.27)) hide)
     )
@@
       (effects (font (size 1.27 1.27)) hide)
     )
-    (property "Manufacturer_Part_Number" "0402WGF4701TCE" (id 4) (at 49.53 267.335 0)
+    (property "Manufacturer_Part_Number" "ERJPA2F4701X" (id 4) (at 49.53 267.335 0)
       (effects (font (size 1.27 1.27)) hide)
     )
@@
       (effects (font (size 1.27 1.27)) hide)
     )
-    (property "Manufacturer_Part_Number" "0402WGF1002TCE" (id 4) (at 35.56 325.12 0)
+    (property "Manufacturer_Part_Number" "RNCF0402BTE10K0" (id 4) (at 35.56 325.12 0)
       (effects (font (size 1.27 1.27)) hide)
     )
@@
       (effects (font (size 1.27 1.27)) hide)
     )
-    (property "Manufacturer_Part_Number" "CL05A225MQ5NSNC" (id 4) (at 16.51 269.875 0)
+    (property "Manufacturer_Part_Number" "ZRB157R61C225KE11D" (id 4) (at 16.51 269.875 0)
       (effects (font (size 1.27 1.27)) hide)
     )
@@
       (effects (font (size 1.27 1.27)) hide)
     )
-    (property "Manufacturer_Part_Number" "0402WGF4701TCE" (id 4) (at 41.91 267.335 0)
+    (property "Manufacturer_Part_Number" "ERJPA2F4701X" (id 4) (at 41.91 267.335 0)
       (effects (font (size 1.27 1.27)) hide)
     )
@@
       (effects (font (size 1.27 1.27)) hide)
     )
-    (property "Manufacturer_Part_Number" "AECR0402F220RK9" (id 4) (at 46.99 226.06 0)
+    (property "Manufacturer_Part_Number" "PTFR0402B220RP9" (id 4) (at 46.99 226.06 0)
       (effects (font (size 1.27 1.27)) hide)
     )
@@
       (effects (font (size 1.27 1.27)) hide)
     )
-    (property "Manufacturer_Part_Number" "0402WGF1002TCE" (id 4) (at 53.34 231.14 0)
+    (property "Manufacturer_Part_Number" "RNCF0402BTE10K0" (id 4) (at 53.34 231.14 0)
       (effects (font (size 1.27 1.27)) hide)
     )
@@
       (effects (font (size 1.27 1.27)) hide)
     )
-    (property "Manufacturer_Part_Number" "0402WGF1002TCE" (id 4) (at 35.56 317.5 0)
+    (property "Manufacturer_Part_Number" "RNCF0402BTE10K0" (id 4) (at 35.56 317.5 0)
       (effects (font (size 1.27 1.27)) hide)
     )
@@
       (effects (font (size 1.27 1.27)) hide)
     )
-    (property "Manufacturer_Part_Number" "0402WGF1002TCE" (id 4) (at 58.42 257.81 0)
+    (property "Manufacturer_Part_Number" "RNCF0402BTE10K0" (id 4) (at 58.42 257.81 0)
       (effects (font (size 1.27 1.27)) hide)
     )
@@
     (in_bom yes) (on_board yes) (fields_autoplaced)
     (property "Reference" "D5" (id 0) (at 58.1025 333.8535 0))
-    (property "Value" "1N5819WS" (id 1) (at 58.1025 336.6286 0))
+    (property "Value" "BAT60JFILM" (id 1) (at 58.1025 336.6286 0))
     (property "Footprint" "Diode_SMD:D_SOD-323" (id 2) (at 58.42 339.09 0)
       (effects (font (size 1.27 1.27)) hide)
@@
       (effects (font (size 1.27 1.27)) hide)
     )
-    (property "Manufacturer_Part_Number" "1N5819WS" (id 4) (at 58.42 339.09 0)
+    (property "Manufacturer_Part_Number" "BAT60JFILM" (id 4) (at 58.42 339.09 0)
       (effects (font (size 1.27 1.27)) hide)
     )
@@
       (effects (font (size 1.27 1.27)) hide)
     )
-    (property "Manufacturer_Part_Number" "CL05A225MQ5NSNC" (id 4) (at 26.67 269.875 0)
-      (effects (font (size 1.27 1.27)) hide)
-    )
+    (property "Manufacturer_Part_Number" "ZRB157R61C225KE11D" (id 4) (at 26.67 269.875 0)
+      (effects (font (size 1.27 1.27)) hide)
+    )
