File: USB_HUB.kicad_sch (KiCad schematic)
At the start: 16 parts

Commit message: плата практически готова
Parts:
- removed R? (x2): 100K, Resistor_SMD:R_0402_1005Metric, symbol Device:R
- removed U? (x2): FSUSB42MUX, Package_DFN_QFN:UQFN-10_1.4x1.8mm_P0.4mm, symbol Interface_USB:FSUSB42MUX
- removed Y?: 24MHz, Crystal:Crystal_SMD_2016-4Pin_2.0x1.6mm, symbol Device:Crystal_GND23
- added C42, C43, C44: 100nF, Capacitor_SMD:C_0402_1005Metric, symbol Device:C
- added R3: 4K7, Resistor_SMD:R_0402_1005Metric, symbol Device:R
- added U14, U18: FSUSB42MUX, Package_DFN_QFN:UQFN-10_1.4x1.8mm_P0.4mm, symbol Interface_USB:FSUSB42MUX
- added Y3: 24MHz, Crystal:Crystal_SMD_2016-4Pin_2.0x1.6mm, symbol Device:Crystal_GND24
- gave numbers to parts that had none: 11
Connections:
- net GND: now also U19.11 (TEST), C42.2, C43.2, C44.2, R3.2, U14.10 (~{OE}), U14.5 (GND), U18.10 (~{OE}), U18.5 (GND), Y3.2, Y3.4
- net USB_BOARD.DN: now also U18.4 (D-)
- net USB_BOARD.DP: now also U18.3 (D+)
- net USB_HUB_3V3: now also C42.1, C43.1, C44.1, U14.1 (VCC), U18.1 (VCC); no longer R49.2, U19.27 (VBUS_DET)
- net USB_RPI.DN: now also U14.4 (D-)
- net USB_RPI.DP: now also U14.3 (D+)
- net USBHUB_SOURCE_DN: now reaches U19.30 (USBDM_UP)
- net USBHUB_SOURCE_DN: now also U14.6 (HSD1-), U18.8 (HSD2-)
- net USBHUB_SOURCE_DP: now reaches U19.31 (USBDP_UP)
- net USBHUB_SOURCE_DP: now also U14.7 (HSD1+), U18.9 (HSD2+)
- net at C21.1, U19.32 (XTALOUT): now also Y3.3
- net at C20.2, U19.33 (XTALIN/CLKIN): now also Y3.1
- net USBHUB_SINK3_DN: now reaches U19.6 (USBDM_DN3/PRT_DIS_M3)
- net USBHUB_SINK3_DN: now also U14.8 (HSD2-), U18.6 (HSD1-)
- net USBHUB_SINK3_DP: now reaches U19.7 (USBDP_DN3/PRT_DIS_P3)
- net USBHUB_SINK3_DP: now also U14.9 (HSD2+), U18.7 (HSD1+)
- net USB_RPI.ID renamed USB_SWITCH
- net USB_SWITCH: now also R3.1, U14.2 (SEL), U18.2 (SEL)
- new net VBUS_SENSE: R49.2, U19.27 (VBUS_DET)
- no-connect marks 11 -> 13
Other:
- moved on the sheet: C20, C21, C22, C23, J7, R48, R49, R51, R52, R53, U19

Commit message: Little fix
Parts:
- C20, C21: Manufacturer_Part_Number (none) -> 0402CG150J500NT
- C22, C23: Manufacturer_Part_Number (none) -> CL05A225MQ5NSNC
- C42, C43, C44: Manufacturer_Part_Number (none) -> CL05B104KB54PNC
- R3: Manufacturer_Part_Number (none) -> 0402WGF4701TCE
- R48, R49, R52, R53: Manufacturer_Part_Number (none) -> 0402WGF100KTCE
- R51: Manufacturer_Part_Number (none) -> RT0402BRD0712K1L
Changed lines of the file:
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@@
+      (effects (font (size 1.27 1.27)) hide)
+    )
+    (property "Manufacturer_Part_Number" "0402WGF100KTCE" (id 4) (at 59.69 124.46 0)
       (effects (font (size 1.27 1.27)) hide)
     )
@@
     )
     (property "Datasheet" "~" (id 3) (at 58.42 72.39 0)
+      (effects (font (size 1.27 1.27)) hide)
+    )
+    (property "Manufacturer_Part_Number" "0402WGF100KTCE" (id 4) (at 58.42 72.39 0)
       (effects (font (size 1.27 1.27)) hide)
     )
@@
       (effects (font (size 1.27 1.27)) hide)
     )
+    (property "Manufacturer_Part_Number" "0402WGF100KTCE" (id 4) (at 53.34 124.46 0)
+      (effects (font (size 1.27 1.27)) hide)
+    )
     (pin "1")
     (pin "2")
@@
       (effects (font (size 1.27 1.27)) hide)
     )
+    (property "Manufacturer_Part_Number" "0402WGF4701TCE" (id 4) (at 209.55 125.73 0)
+      (effects (font (size 1.27 1.27)) hide)
+    )
     (pin "1")
     (pin "2")
@@
       (effects (font (size 1.27 1.27)) hide)
     )
+    (property "Manufacturer_Part_Number" "0402WGF100KTCE" (id 4) (at 62.23 124.46 0)
+      (effects (font (size 1.27 1.27)) hide)
+    )
     (pin "1")
     (pin "2")
@@
       (effects (font (size 1.27 1.27)) hide)
     )
+    (property "Manufacturer_Part_Number" "CL05A225MQ5NSNC" (id 4) (at 113.03 36.83 0)
+      (effects (font (size 1.27 1.27)) hide)
+    )
     (pin "1")
     (pin "2")
@@
     )
     (property "Datasheet" "~" (id 3) (at 44.45 109.22 0)
+      (effects (font (size 1.27 1.27)) hide)
+    )
+    (property "Manufacturer_Part_Number" "0402CG150J500NT" (id 4) (at 44.45 109.22 0)
       (effects (font (size 1.27 1.27)) hide)
     )
@@
       (effects (font (size 1.27 1.27)) hide)
     )
+    (property "Manufacturer_Part_Number" "CL05B104KB54PNC" (id 4) (at 146.05 36.83 0)
+      (effects (font (size 1.27 1.27)) hide)
+    )
     (pin "1")
     (pin "2")
@@
       (effects (font (size 1.27 1.27)) hide)
     )
+    (property "Manufacturer_Part_Number" "CL05A225MQ5NSNC" (id 4) (at 102.87 36.83 0)
+      (effects (font (size 1.27 1.27)) hide)
+    )
     (pin "1")
     (pin "2")
@@
     )
     (property "Datasheet" "~" (id 3) (at 31.75 109.22 0)
+      (effects (font (size 1.27 1.27)) hide)
+    )
+    (property "Manufacturer_Part_Number" "0402CG150J500NT" (id 4) (at 31.75 109.22 0)
       (effects (font (size 1.27 1.27)) hide)
     )
@@
     )
     (property "Datasheet" "~" (id 3) (at 58.42 80.01 0)
+      (effects (font (size 1.27 1.27)) hide)
+    )
+    (property "Manufacturer_Part_Number" "RT0402BRD0712K1L" (id 4) (at 58.42 80.01 0)
       (effects (font (size 1.27 1.27)) hide)
     )
@@
       (effects (font (size 1.27 1.27)) hide)
     )
+    (property "Manufacturer_Part_Number" "CL05B104KB54PNC" (id 4) (at 134.62 36.83 0)
+      (effects (font (size 1.27 1.27)) hide)
+    )
     (pin "1")
     (pin "2")
@@
       (effects (font (size 1.27 1.27)) hide)
     )
+    (property "Manufacturer_Part_Number" "CL05B104KB54PNC" (id 4) (at 123.19 36.83 0)
+      (effects (font (size 1.27 1.27)) hide)
+    )

Commit message: First order
Parts:
- C20, C21: Manufacturer_Part_Number 0402CG150J500NT -> GJM1555C1H150GB01D
- C22, C23: Manufacturer_Part_Number CL05A225MQ5NSNC -> ZRB157R61C225KE11D
- C42, C43, C44: Manufacturer_Part_Number CL05B104KB54PNC -> C1005X7R1H104KT000S
- R3: Manufacturer_Part_Number 0402WGF4701TCE -> ERJPA2F4701X
- R48, R49, R52, R53: Manufacturer_Part_Number 0402WGF100KTCE -> PTFR0402B100KN9
- R51: Manufacturer_Part_Number RT0402BRD0712K1L -> RN731ETTP1202B25
Changed lines of the file:
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@@
       (effects (font (size 1.27 1.27)) hide)
     )
-    (property "Manufacturer_Part_Number" "0402WGF100KTCE" (id 4) (at 59.69 124.46 0)
+    (property "Manufacturer_Part_Number" "PTFR0402B100KN9" (id 4) (at 59.69 124.46 0)
       (effects (font (size 1.27 1.27)) hide)
     )
@@
       (effects (font (size 1.27 1.27)) hide)
     )
-    (property "Manufacturer_Part_Number" "0402WGF100KTCE" (id 4) (at 58.42 72.39 0)
+    (property "Manufacturer_Part_Number" "PTFR0402B100KN9" (id 4) (at 58.42 72.39 0)
       (effects (font (size 1.27 1.27)) hide)
     )
@@
       (effects (font (size 1.27 1.27)) hide)
     )
-    (property "Manufacturer_Part_Number" "0402WGF100KTCE" (id 4) (at 53.34 124.46 0)
+    (property "Manufacturer_Part_Number" "PTFR0402B100KN9" (id 4) (at 53.34 124.46 0)
       (effects (font (size 1.27 1.27)) hide)
     )
@@
       (effects (font (size 1.27 1.27)) hide)
     )
-    (property "Manufacturer_Part_Number" "0402WGF4701TCE" (id 4) (at 209.55 125.73 0)
+    (property "Manufacturer_Part_Number" "ERJPA2F4701X" (id 4) (at 209.55 125.73 0)
       (effects (font (size 1.27 1.27)) hide)
     )
@@
       (effects (font (size 1.27 1.27)) hide)
     )
-    (property "Manufacturer_Part_Number" "0402WGF100KTCE" (id 4) (at 62.23 124.46 0)
+    (property "Manufacturer_Part_Number" "PTFR0402B100KN9" (id 4) (at 62.23 124.46 0)
       (effects (font (size 1.27 1.27)) hide)
     )
@@
       (effects (font (size 1.27 1.27)) hide)
     )
-    (property "Manufacturer_Part_Number" "CL05A225MQ5NSNC" (id 4) (at 113.03 36.83 0)
+    (property "Manufacturer_Part_Number" "ZRB157R61C225KE11D" (id 4) (at 113.03 36.83 0)
       (effects (font (size 1.27 1.27)) hide)
     )
@@
       (effects (font (size 1.27 1.27)) hide)
     )
-    (property "Manufacturer_Part_Number" "0402CG150J500NT" (id 4) (at 44.45 109.22 0)
+    (property "Manufacturer_Part_Number" "GJM1555C1H150GB01D" (id 4) (at 44.45 109.22 0)
       (effects (font (size 1.27 1.27)) hide)
     )
@@
       (effects (font (size 1.27 1.27)) hide)
     )
-    (property "Manufacturer_Part_Number" "CL05B104KB54PNC" (id 4) (at 146.05 36.83 0)
+    (property "Manufacturer_Part_Number" "C1005X7R1H104KT000S" (id 4) (at 146.05 36.83 0)
       (effects (font (size 1.27 1.27)) hide)
     )
@@
       (effects (font (size 1.27 1.27)) hide)
     )
-    (property "Manufacturer_Part_Number" "CL05A225MQ5NSNC" (id 4) (at 102.87 36.83 0)
+    (property "Manufacturer_Part_Number" "ZRB157R61C225KE11D" (id 4) (at 102.87 36.83 0)
       (effects (font (size 1.27 1.27)) hide)
     )
@@
       (effects (font (size 1.27 1.27)) hide)
     )
-    (property "Manufacturer_Part_Number" "0402CG150J500NT" (id 4) (at 31.75 109.22 0)
+    (property "Manufacturer_Part_Number" "GJM1555C1H150GB01D" (id 4) (at 31.75 109.22 0)
       (effects (font (size 1.27 1.27)) hide)
     )
@@
       (effects (font (size 1.27 1.27)) hide)
     )
-    (property "Manufacturer_Part_Number" "RT0402BRD0712K1L" (id 4) (at 58.42 80.01 0)
+    (property "Manufacturer_Part_Number" "RN731ETTP1202B25" (id 4) (at 58.42 80.01 0)
       (effects (font (size 1.27 1.27)) hide)
     )
@@
       (effects (font (size 1.27 1.27)) hide)
     )
-    (property "Manufacturer_Part_Number" "CL05B104KB54PNC" (id 4) (at 134.62 36.83 0)
+    (property "Manufacturer_Part_Number" "C1005X7R1H104KT000S" (id 4) (at 134.62 36.83 0)
       (effects (font (size 1.27 1.27)) hide)
     )
@@
       (effects (font (size 1.27 1.27)) hide)
     )
-    (property "Manufacturer_Part_Number" "CL05B104KB54PNC" (id 4) (at 123.19 36.83 0)
-      (effects (font (size 1.27 1.27)) hide)
-    )
+    (property "Manufacturer_Part_Number" "C1005X7R1H104KT000S" (id 4) (at 123.19 36.83 0)
+      (effects (font (size 1.27 1.27)) hide)
+    )
